File: interface/Designs/OOBDtiger/ARM_CortexA8_DEBIAN/D5/pcb/OOBD-TigerV2.sch (EAGLE design)
At the start: 65 parts, among them U1 SY6280, U10 MP1482DS, U2 SN65HVD230(SO8), U6 SN65HVD230(SO8)

Commit message: Verzeichnis enhaelt jetzt noch die Schematics & PCB von Audiocape und die aktualisierten Dateien von OOBD-Tiger V2. Im Moment in das falsche IC TLV320AIC3104. Housing und Package vom TLV320AIC3107 müssen noch erzeugt werden, lib dazu habe ich nicht fertig gefunden. Werde das 04 als Vorlage nehmen.
Parts:
- removed CAN, CAN1: TB3-3.5mm, DOUBLE-SIDE:CON33.5MM
- removed FID1, FID2, FID3: FIDUCIAL, SparkFunEagle-6-6-07:FIDUCIAL
- added C10, C11, C16, C17, C8, C9: 0.1uf, SparkFun-Passives:CAP0402-CAP
- added C12, C13, C14, C15: 10uf,10V, SparkFun-Passives:CAP0603-CAP
- added C18, C19, C5, C7: 47pF, SparkFun-Passives:CAP0402-CAP
- added C2, C3: 47uf, SparkFun-Capacitors:CAP_POL1206
- added C20: 1uf, SparkFun-Passives:CAP0402-CAP
- added C21: .01uf, SparkFun-Passives:CAP0402-CAP
- added C22: 2.2uf, SparkFun-Passives:CAP0402-CAP
- added D1, D2, D3, D5: PGB0010603MR, CircuitCo:PGB0010603MR
- added FB1, FB2: FB, SparkFun-Passives:FB
- added J2, U$3: SJ1-3515-SMT-TR, audio-jack:SJ1-3515-SMT-TR
- added J3: (no value), SparkFun-Connectors:M04PTH
- added K1: 653112124022, EagleLibrary_Wuerth_Elektronik _eiCan_Wire_to_Board_Connectors_v6_20150113:653112124022
- added R10, R11: 0, SparkFun-Passives:RESISTOR0805-RES
- added R8, R9: 33, SparkFun-Passives:RESISTOR0402-RES
- added U3: V_REG_LDOSMD, SparkFun-PowerIC:V_REG_LDOSMD
- added U4: TLV320AIC3104, CircuitCo:TLV320AIC3104
- C51: device rcl:CPOL-EUE5-10.5 -> rcl:CPOL-EUE3.5-8
Connections:
- new net 1.8V: C11.1, C15.2, C22.1, U3.OUT, U4.DVDD
- new net 3.3V: C10.1, C14.2, C20.1, FB2.P$2, U3.EN, U3.IN, U4.IOVDD
- new net AGND: C12.1, C13.1, C18.2, C19.1, C5.2, C7.2, C8.2, C9.2, D1.P$1, D2.P$1, D3.P$1, D5.P$1, FB1.P$1, J2.1, U$3.1, U4.AVSS_ADC, U4.AVSS_DAC
- new net AUD_3V3: C12.2, C13.2, C8.1, C9.1, FB2.P$1, U4.AVDD_DAC, U4.DRVDD, U4.DRVDD2
- new net AUD_BCLK: U4.BCLK
- new net AUD_DIN: U4.DOUT
- new net AUD_DOUT: U4.DIN
- new net AUD_HPLOUT: C2.+, R10.2, U4.HPLOUT
- new net AUD_HPROUT: C3.+, R11.2, U4.HPROUT
- new net AUD_MCLK: U4.MCLK
- new net AUD_WCLK: U4.WCLK
- new net DGND: C10.2, C11.2, C14.1, C15.1, C20.2, C21.2, C22.2, FB1.P$2, U3.GND, U4.DRVSS, U4.DVSS, U4.PAD
- new net J1: C7.1, D2.P$2, R8.1, U$3.2
- new net LEFT_LOM: J3.1, U4.LEFT_LOM
- new net LEFT_LOP: J3.2, U4.LEFT_LOP
- new net LINE1LP: C16.2, U4.IN2L
- new net LINE1RP: C17.1, U4.IN2R
- new net N$10: C2.-, R10.1, R8.2
- new net N$14: C3.-, R11.1, R9.2
- new net N$15: C5.1, D1.P$2, R9.1, U$3.3
- new net N$16: C17.2, C19.2, D3.P$2, J2.3
- new net N$17: C16.1, C18.1, D5.P$2, J2.2
- new net N$18: C21.1, U3.BP
- new net RESETN: U4.RESETN
- new net RIGHT_LOP: J3.4, U4.RIGHT_LOP
- new net RIGHT_ROM: J3.3, U4.RIGHT_ROM
- new net SCL: U4.SCL
- new net SDA: U4.SDA
- net CANH: now also K1.5; no longer CAN.3
- net CANH1: now also K1.1; no longer CAN1.3
- net CANL: now also K1.7; no longer CAN.2
- net CANL1: now also K1.3; no longer CAN1.2
- net GND: now also K1.4; no longer CAN.1, CAN1.1
Other:
- note added: "Audio"
- note added: "HS CAN DRIVER"
- note added: "MS CAN DRIVER"
- note removed: "CAN DRIVER"
- moved on the sheet: 5V_E, AM3352-SOM-EVB-PLATFORM, C1, C4, C47, C48, C49, C50, C51, C52, C53, C54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
