File: interface/Designs/OOBDtiger/ARM_CortexA8_DEBIAN/D5/pcb/OOBD-TigerV2.sch (EAGLE design)
At the start: 81 parts, among them K1 653112124022, U1 SY6280, U10 MP1482DS, U2 SN65HVD230(SO8), U6 SN65HVD230(SO8)

Commit message: Modifications on OOBD-Tiger schematics: - separate physical blocks (CAN, USB, Connectors, Ausio, Power Supply) to different pages - delete unneeded parts (so far) - replace OBD2-Interface connector to OOBD CAN Invader Interface
Parts:
- removed CAN1_RX/CAN0_RX, CAN1_RX/CAN0_RX1: HN1x3(CAN1_RX:Close/CAN0_RX:Open), jumper:JP2E
- removed CAN1_TX/CAN0_TX, CAN1_TX/CAN0_TX1: HN1x3(CAN1_TX:Close/CAN0_TX:Open), jumper:JP2E
- removed GND_PIN: TESTPAD3, gogo:TESTPAD3
- removed K1: 653112124022, EagleLibrary_Wuerth_Elektronik _eiCan_Wire_to_Board_Connectors_v6_20150113:653112124022
- removed PWR: YDJ-1136, gogo:PWR-JAKPWR_JACK_UNI_MILLING
- removed USB_PWR_E: HN1x2(Open), jumper:JP1E
- added OBD2-CONNECTOR: (no value), pinhead:PINHD-2X5/90
Connections:
- removed net CAN_RX: CAN1_RX/CAN0_RX.2, CAN1_RX/CAN0_RX1.2, U2.RXD, U6.RXD
- removed net CAN_TX: CAN1_TX/CAN0_TX.2, CAN1_TX/CAN0_TX1.2, U2.TXD, U6.TXD
- removed net N$3: C51.+, D4.C, PWR.+, R69.1, U10.IN
- removed net P2_9/LCD_D3: AM3352-SOM-EVB-PLATFORM.P2_9/LCD_D3
- new net +12V: C51.+, D4.C, OBD2-CONNECTOR.10, R69.1, U10.IN
- net +5V: no longer USB_PWR_E.2
- net +5V_OTG_PWR: no longer USB_PWR_E.1
- net CANH: now also OBD2-CONNECTOR.1; no longer K1.5
- net CANH1: now also OBD2-CONNECTOR.7; no longer K1.1
- net CANL: now also OBD2-CONNECTOR.2; no longer K1.7
- net CANL1: now also OBD2-CONNECTOR.6; no longer K1.3
- net GND: now also OBD2-CONNECTOR.3; no longer GND_PIN.PP, K1.4, PWR.-, PWR.--
- net P0_12/I2C2_SDA: now also U6.TXD; no longer CAN1_TX/CAN0_TX.1, CAN1_TX/CAN0_TX1.1
- net P0_13/I2C2_SCL: now also U6.RXD; no longer CAN1_RX/CAN0_RX.1, CAN1_RX/CAN0_RX1.1
- net P1_8/UART4_RXD: now also U2.TXD; no longer CAN1_TX/CAN0_TX.3, CAN1_TX/CAN0_TX1.3
- net P1_9/UART4_TXD: now also U2.RXD; no longer CAN1_RX/CAN0_RX.3, CAN1_RX/CAN0_RX1.3
Other:
- note added: "Author: W. Sauer, M. Luxen"
- note added: "OBD2-Power supply"
- note added: "Power Supply (6-16V)"
- note added: "Project: OOBD-Tiger"
- note added: "Title: Audio"
- note added: "Title: CAN-Interfaces"
- note added: "Title: Connector for AM3352SOM"
- note added: "Title: Power Supply"
- note added: "Title: USB-Interfaces (OTG / HOST)"
- note removed: "6-16VDC"
- note removed: "Power Supply"
