File: interface/Designs/OOBDtiger/ARM_CortexA8_DEBIAN/D5/pcb/OOBD-TigerV2.brd (EAGLE design)
At the start: 63.4 x 38.2 mm, 81 parts, among them K1 653112124022, U1 SY6280, U10 MP1482DS, U2 SN65HVD230(SO8), U6 SN65HVD230(SO8)

Commit message: Modifications on OOBD-Tiger schematics: - separate physical blocks (CAN, USB, Connectors, Ausio, Power Supply) to different pages - delete unneeded parts (so far) - replace OBD2-Interface connector to OOBD CAN Invader Interface
Parts:
- removed CAN1_RX/CAN0_RX, CAN1_RX/CAN0_RX1: HN1x3(CAN1_RX:Close/CAN0_RX:Open), jumper:JP2
- removed CAN1_TX/CAN0_TX, CAN1_TX/CAN0_TX1: HN1x3(CAN1_TX:Close/CAN0_TX:Open), jumper:JP2
- removed GND_PIN: TESTPAD3, gogo:TEST_PAD40/70/SQUARE
- removed K1: 653112124022, EagleLibrary_Wuerth_Elektronik _eiCan_Wire_to_Board_Connectors_v6_20150113:653112124022
- removed PWR: YDJ-1136, gogo:PWR_JACK_UNI_MILLING
- removed USB_PWR_E: HN1x2(Open), jumper:JP1
- added OBD2-CONNECTOR: (no value), pinhead:2X05/90
Connections:
- removed net CAN_RX: CAN1_RX/CAN0_RX.2, CAN1_RX/CAN0_RX1.2, U2.4, U6.4
- removed net CAN_TX: CAN1_TX/CAN0_TX.2, CAN1_TX/CAN0_TX1.2, U2.1, U6.1
- removed net N$3: C51.+, D4.C, PWR.+, R69.1, U10.2
- removed net P2_9/LCD_D3: AM3352-SOM-EVB-PLATFORM.1-11
- new net +12V: C51.+, D4.C, OBD2-CONNECTOR.10, R69.1, U10.2
- net +5V: no longer USB_PWR_E.2
- net +5V_OTG_PWR: no longer USB_PWR_E.1
- net CANH: now also OBD2-CONNECTOR.1; no longer K1.5
- net CANH1: now also OBD2-CONNECTOR.7; no longer K1.1
- net CANL: now also OBD2-CONNECTOR.2; no longer K1.7
- net CANL1: now also OBD2-CONNECTOR.6; no longer K1.3
- net GND: now also OBD2-CONNECTOR.3; no longer GND_PIN.P$1, K1.4, PWR.-, PWR.--
- net P0_12/I2C2_SDA: now also U6.1; no longer CAN1_TX/CAN0_TX.1, CAN1_TX/CAN0_TX1.1
- net P0_13/I2C2_SCL: now also U6.4; no longer CAN1_RX/CAN0_RX.1, CAN1_RX/CAN0_RX1.1
- net P1_8/UART4_RXD: now also U2.1; no longer CAN1_TX/CAN0_TX.3, CAN1_TX/CAN0_TX1.3
- net P1_9/UART4_TXD: now also U2.4; no longer CAN1_RX/CAN0_RX.3, CAN1_RX/CAN0_RX1.3
Routing:
- net N$3: track 110.4 -> 0.00 mm, vias 3 -> 0
- net +12V: track 0.00 -> 110.4 mm, vias 0 -> 3
- net CAN_TX: track 53.2 -> 0.00 mm, vias 1 -> 0
- net CAN_RX: track 52.4 -> 0.00 mm, vias 5 -> 0
- net P1_8/UART4_RXD: track 34.1 -> 22.1 mm
- net P0_12/I2C2_SDA: track 31.7 -> 22.2 mm
- net P1_9/UART4_TXD: track 24.9 -> 16.4 mm
- net +5V_OTG_PWR: track 66.6 -> 62.8 mm
- net +5V: track 142.0 -> 139.3 mm
- net P0_13/I2C2_SCL: track 32.0 -> 29.4 mm
- net GND: track 279.5 -> 277.8 mm
