File: interface/Designs/OOBDtiger/ARM_CortexA8_DEBIAN/D5/pcb/OOBD-Tiger.brd (EAGLE design)
At the start: 63.4 x 38.2 mm, 88 parts, among them IC3 DS1307, IC4 DS3231, Q2 32.768kHz, U1 SY6280, U10 MP1482DS, U2 SN65HVD230(SO8), U6 SN65HVD230(SO8)

Commit message: - delete unneeded nets - connect DCAN0, DCAN1, RTC und Audio to AM3352 GPIO (X-Check necessary) - minor cosmetic stuff
Other:
- board text removed: "+"
- board text removed: "+5V"
- board text removed: "-"
- board text removed: "1"
- board text removed: "10"
- board text removed: "11"
- board text removed: "12"
- board text removed: "13"
- board text removed: "14"
- board text removed: "15"
- board text removed: "16"
- board text removed: "17"
- board text removed: "18"
- board text removed: "19"
- board text removed: "2"
- board text removed: "20"
- board text removed: "21"
- board text removed: "22"
- board text removed: "23"
- board text removed: "24"
- board text removed: "25"
- board text removed: "26"
- board text removed: "27"
- board text removed: "28"
- board text removed: "29"
- board text removed: "3"
- board text removed: "30"
- board text removed: "31"
- board text removed: "32"
- board text removed: "33"
- board text removed: "34"
- board text removed: "35"
- board text removed: "36"
- board text removed: "37"
- board text removed: "38"
- board text removed: "39"
- board text removed: "4"
- board text removed: "40"
- board text removed: "5"
- board text removed: "5V power supply is disabled"
- board text removed: "5V power supply is enabled (default)"
- board text removed: "5V_E"
- board text removed: "6"
- board text removed: "6-16VDC"
- board text removed: "7"
- board text removed: "8"
- board text removed: "9"
- board text removed: "AM3352-SOM-EVB"
- board text removed: "CAN0 is selected"
- board text removed: "CAN1 is selected (default)"
- board text removed: "CAN1_RX/CAN0_RX"
- board text removed: "CAN1_TX/CAN0_TX"
- board text removed: "CAN_H"
- board text removed: "CAN_L"
- board text removed: "CAN_T"
- board text removed: "CAN_T is disabled (default)"
- board text removed: "CAN_T is enabled"
- board text removed: "D+"
- board text removed: "D-"
- board text removed: "DESCRIPTION"
- board text removed: "GND"
- board text removed: "HOST_DRV"
- board text removed: "JUMPER"
- board text removed: "RX"
- board text removed: "Rev.D"
- board text removed: "STATE"
- board text removed: "TX"
- board text removed: "USB power supply is disabled (default)"
- board text removed: "USB power supply is enabled"
- board text removed: "USB1_DRV is disabled"
- board text removed: "USB1_DRV is enabled (default)"
- board text removed: "USB_PWR_E"
