File: interface/Designs/OOBDtiger/ARM_CortexA8_DEBIAN/D5/pcb/OOBD-Tiger.brd (EAGLE design)
At the start: 63.4 x 38.2 mm, 136 parts, among them IC1 ADM3053M, IC2 ADM3053M, IC4 DS3231, U1 SY6280, U10 MP1482DS, U2 SN65HVD230(SO8), U3 SY6280, U4 TLV70215, U6 SN65HVD230(SO8)

Commit message: modifications after schematics review
Parts:
- removed L4: FB0805/600R/2A, rcl:L0603
- removed R10, R11, R12, R15, R16, R17, R18: 0, resistor:R0603
- removed SPEAKER: LS1, SparkFun:1X02
- added JP2: Audio-Out, jumper:JP3Q
- added L2: FB0805/600R/200mA(201209-601), rcl:L0603
- added R34, R35: 0R, rcl:R0603
- C18, C19: value 0,01µF -> NI (0,01µF)
- C22, C26, C28, C30: value 10µF -> 10nF
- C31: value NA (AY2221K29Y5SS63L7) -> NI (AY2221K29Y5SS63L7)
- C37: value NA (47pF) -> NI (47pF)
- C38: value 1.0µF -> 0.1nF
- C44: value 1.0µF -> 10µF
- OOBDPICAN: value Bridge to PICAN -> Bridge to OOBDpiCAN
- R13, R14: value 0 -> 0R; device resistor:R0603 -> resistor:R0805
- R2, R23, R40, R55, R7: value NA -> NI
- U10: value MP1482DS -> MP1482
- moved C43 36.4 mm to (2.54, -4.45)
- moved C44 32.7 mm to (12.7, -5.08)
- moved C42 31.7 mm to (2.54, -1.27)
- moved C40 28.9 mm to (12.7, -2.54)
- moved C41 28.4 mm to (7.62, -3.17)
- moved C45 27.2 mm to (17.8, -5.71), turned to 0 degrees
- moved C57 26.7 mm to (30.5, -6.99), turned to 0 degrees
- moved C39 26.2 mm to (17.8, -1.91)
- moved C46 19.7 mm to (22.9, -6.35), turned to 0 degrees
- moved C9 6.73 mm to (31.4, 34.9), turned to 180 degrees
- moved R3 3.98 mm to (10.2, 33.0), turned to 270 degrees
- moved R5 3.14 mm to (36.2, 34.9)
- moved C49 2.48 mm to (7.62, 12.7), turned to 270 degrees
- moved D4 2.25 mm to (11.4, 15.9)
- moved L11 1.93 mm to (12.7, 19.7)
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Connections:
- net CAN0_H renamed MS-CAN_H
- net CAN1_H renamed HS-CAN_H
- removed net CAN0_L: D1.1, IC2.15, MS-CAN.2, OOBD2-CONNECTOR.2, R28.1
- removed net CAN1_L: D2.1, HS-CAN.2, IC1.15, OOBD2-CONNECTOR.6, R30.1
- removed net GND1: C45.1, C46.1
- removed net N$20: R12.1, TLV320AIC3107.29
- removed net N$21: C45.2, C46.2, TLV320AIC3107.40
- removed net N$22: R17.2, TLV320AIC3107.38
- removed net N$23: R16.2, TLV320AIC3107.37
- removed net N$24: R15.2, TLV320AIC3107.35
- removed net N$25: R10.2, TLV320AIC3107.36
- removed net N$26: R18.2, TLV320AIC3107.34
- new net HS-CAN_L: D2.1, HS-CAN.1, IC1.15, OOBD2-CONNECTOR.6, R30.1
- new net MS-CAN_L: D1.1, IC2.15, MS-CAN.1, OOBD2-CONNECTOR.2, R28.1
- new net N$17: R14.1, TLV320AIC3107.26
- new net USB0_EN: R2.1, R34.1, R4.2, U1.4
- new net USB1_EN: R21.2, R23.1, R35.1, U3.4
- net +3V3: now also C27.1, C28.1, C29.1, C30.1, C39.2, C40.2, C45.2, C46.2, IC1.6, IC2.6, TLV320AIC3107.40; no longer C11.1, C12.1, C13.1, C14.1, C39.1, C40.1, IC1.8, IC2.8
- net +5V: now also C11.1, C12.1, C13.1, C14.1, IC1.8, IC2.8; no longer C27.1, C28.1, C29.1, C30.1, IC1.6, IC2.6
- net AGND: now also C18.1, JP2.5, L2.2, TLV320AIC3107.27, TLV320AIC3107.30; no longer C18.2
- net AUD_BCLK: now also TLV320AIC3107.35; no longer R15.1
- net AUD_DIN: now also TLV320AIC3107.38; no longer R16.1
- net AUD_DOUT: now also TLV320AIC3107.37; no longer R17.1
- net AUD_MCLK: now also TLV320AIC3107.34; no longer R18.1
- net AUD_WCLK: now also TLV320AIC3107.36; no longer R10.1
- net GND: now also C39.1, C40.1, C45.1, C46.1, JP2.6, L2.1; no longer C39.2, C40.2, R12.2, R14.1, TLV320AIC3107.26
- net N$14: now also JP2.1, TLV320AIC3107.20; no longer C19.2, L4.2, R14.2
- net N$15: now also C18.2, JP2.4; no longer C18.1, SPEAKER.2
- net N$16: now also C19.2, JP2.2, R14.2; no longer L4.1, SPEAKER.1
- net N$18: no longer R11.2
- net N$19: now also JP2.3, TLV320AIC3107.19; no longer R11.1, TLV320AIC3107.28
- net N$30: now also HS-CAN.2; no longer HS-CAN.1
- net N$32: now also MS-CAN.2; no longer MS-CAN.1
- net USB0_DRV: now also R34.2; no longer R2.1, R4.2, U1.4
- net USB1_DRV: now also R35.2; no longer R21.2, R23.1, U3.4
Routing:
- net GND: track 439.1 -> 0.00 mm, vias 18 -> 0
- net +5V: track 172.9 -> 0.00 mm, vias 12 -> 0
- net +3V3: track 145.5 -> 0.00 mm, vias 15 -> 0
- net GNDA: track 107.3 -> 0.00 mm, vias 5 -> 0
- net USB0_DRV: track 101.1 -> 0.00 mm, vias 4 -> 0
- net +12V: track 97.9 -> 0.00 mm, vias 3 -> 0
- net USB0_DP: track 96.3 -> 0.00 mm, vias 1 -> 0
- net USB1_DRV: track 78.8 -> 0.00 mm
- net USB1_DP: track 77.8 -> 0.00 mm, vias 2 -> 0
- net USB0_ID: track 77.6 -> 0.00 mm, vias 3 -> 0
- net USB1_VBUS: track 74.6 -> 0.00 mm, vias 2 -> 0
- net USB1_ID: track 72.0 -> 0.00 mm, vias 5 -> 0
- net USB0_VBUS: track 70.3 -> 0.00 mm, vias 2 -> 0
- net USB0_DM: track 68.7 -> 0.00 mm, vias 5 -> 0
- net USB0_CE: track 68.4 -> 0.00 mm, vias 4 -> 0
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
Commit message: add minor changes in schematics and optimize placing of parts on OOBD-Tiger PCB
Parts:
- removed C63, C64: 22uF/6.3V, rcl:C0603
- removed L11: 10uH/3.15A/20%, OLIMEX_DISCRET:8X8MM_3131
- removed R47, R48, R49, R84, R86: 2.2k/1%, rcl:R0603
- removed R54: 49.9R/1%, rcl:R0603
- removed R55: NI, rcl:R0603
- removed R69: 10k, rcl:R0603
- removed R70: 4.99k/1%, rcl:R0603
- removed R85: 1.05k/1%, rcl:R0603
- added C58: NI (47pF), SparkFun-Passives:0603-CAP
- added C59: 2.2µf, SparkFun-Passives:0603-CAP
- added L4: FB0805/600R/2A, rcl:L0603
- added R10: 60R, resistor:R0603
- added R11: NI, rcl:R0603
- added R12, R17, R18: 10k, rcl:R0603
- added R15: 13k/1%, rcl:R0603
- added R16: 6k8k/1%, rcl:R0603
- added R36: 1.05k/1%, rcl:R0603
- added R37: 4.99k/1%, rcl:R0603
- added R38, R39: 2.2k/1%, rcl:R0603
- C10, C8: value 22uF/6.3V -> 100nF; device rcl:C0603 -> rcl:C0603K
- C12, C24: value 10µF -> 100nF; device rcl:C0805K -> rcl:C0603K
- C13, C2: value 100nF -> 10µF; device rcl:C0603K -> rcl:C0805K
- C14: value 10µF -> NI (10nF); device rcl:C0805K -> resistor:C0603
- C16, C5: value 0.1µF -> 10nF; device SparkFun-Passives:0603-CAP -> rcl:C0805K
- C17: value 10µF -> NI (AY2221K29Y5SS63L7); device SparkFun-Passives:0603-CAP -> rcl:C075-032X103
- C18: value NI (0,01µF) -> 100nF; device SparkFun-Passives:0603-CAP -> rcl:C0603K
- C19: value NI (0,01µF) -> 10µF; device SparkFun-Passives:0603-CAP -> rcl:C0805K
- C20: value 10µF -> 10nF
- C22, C30: value 10nF -> 100nF; device rcl:C0805K -> rcl:C0603K
- C25, C27: value 100nF -> 22uF/6.3V; device rcl:C0603K -> rcl:C0603
- C26, C28: value 10nF -> 22uF/6.3V; device rcl:C0805K -> rcl:C0603
- C3: value 100nF -> NI (10nF); device rcl:C0603K -> resistor:C0603
- C31: value NI (AY2221K29Y5SS63L7) -> 10µF; device rcl:C075-032X103 -> SparkFun-Passives:0603-CAP
- C32: value NA (AY2221K29Y5SS63L7) -> 0.1µF; device rcl:C075-032X103 -> SparkFun-Passives:0603-CAP
- C33: value NA(10nF) -> 10µF; device resistor:C0603 -> SparkFun-Passives:0603-CAP
- C34: value NA(10nF) -> 0.1µF; device resistor:C0603 -> SparkFun-Passives:0603-CAP
- C35: value 1µf -> 10µF
- C36: value 2.2µf -> 0.1µF
- C37: value NI (47pF) -> 10µF
- C39: value 0.1µF -> 22µF
- C40, C43, C44: value 10µF -> 0.1µF
- C41: value 0.1µF -> 10µF
- C45: value 0.1µF -> NI (0,01µF)
- C46: value 10µF -> NI (0,01µF)
- C47: value 100nF -> 1uF; device rcl:C0603K -> rcl:C0603
- C48: value 100nF -> 470uF/25V/LOWESR/105C; device rcl:C0603 -> SparkFun-Capacitors:PANASONIC_D
- C49: value 10nF -> 100nF
- C50: value 3.3nF -> 100nF
- C51: value 470uF/25V/LOWESR/105C -> 10nF; device SparkFun-Capacitors:PANASONIC_D -> rcl:C0603
- C52: value 100nF -> 3.3nF
- C57: value 0.1µF -> 1µf
- C6: value 100nF -> NI (AY2221K29Y5SS63L7); device rcl:C0603K -> rcl:C075-032X103
- C7: value 22µF -> 10µF; device SparkFun-Passives:0603-CAP -> rcl:C0805K
- C9: value 1uF -> 10nF; device rcl:C0603 -> rcl:C0805K
- L1, L5: value FB0805/600R/2A -> FB0805/600R/200mA(201209-601)
- L2, L3: value FB0805/600R/200mA(201209-601) -> FB0805/600R/2A
- L6: value FB0805/600R/2A -> 10uH/3.15A/20%; device rcl:L0603 -> OLIMEX_DISCRET:8X8MM_3131
- R1: value 2.2k/1% -> 8k2
- R13, R14: device resistor:R0805 -> rcl:0207/10
- R19: value 6k8k/1% -> 10k/1%
- R2: value NI -> 60R; device rcl:R0603 -> resistor:R0603
- R20: value 10k -> 2.2k/1%
- R21, R4: value 10k -> NI
- R22: value 2.2k/1% -> 0R
- R23, R40: value NI -> 2.2k/1%
- R24: value 10k/1% -> NI
- R25: value 8k2 -> 0R
- R26: value 8k2 -> 10K; device rcl:R0603 -> resistor:R0603
- R27: value 0R -> 10K; device rcl:0207/10 -> resistor:R0603
- R28, R29: device rcl:0207/10 -> resistor:R0805
- R3: value 13k/1% -> 60R; device rcl:R0603 -> resistor:R0603
- R30: value 0R -> 2.2k/1%; device rcl:0207/10 -> rcl:R0603
- R31: value 60R -> NI; device resistor:R0603 -> rcl:R0603
- R32, R33: value 60R -> 10k; device resistor:R0603 -> rcl:R0603
- R34: value 0R -> 49.9R/1%
- R35: value 0R -> 2.2k/1%
- R41: value 10k -> 0R; device rcl:R0603 -> rcl:0207/10
- R6: value 60R -> 0R; device resistor:R0603 -> rcl:0207/10
- R7: value NI -> 0R; device rcl:R0603 -> rcl:0207/10
- R8: value 10K -> 8k2; device resistor:R0603 -> rcl:R0603
- R9: value 10K -> 60R
- U1: value SY6280 -> SN65HVD230(SO8); device OLIMEX_IC:SOT23-5 -> arm:SO-08
- U4: value TLV70215 -> SY6280; device SparkFun-PowerIC:SOT23-5 -> OLIMEX_IC:SOT23-5
- U6: value SN65HVD230(SO8) -> TLV70215; device arm:SO-08 -> SparkFun-PowerIC:SOT23-5
- moved C3 55.8 mm to (56.8, 36.5)
- moved R1 53.4 mm to (55.9, 21.6), turned to 180 degrees
- moved C24 51.8 mm to (5.08, 23.5), turned to 90 degrees
- moved C25 51.3 mm to (3.49, 29.8), turned to 180 degrees
- moved R9 49.4 mm to (62.2, 36.2), flipped to the top, turned to 270 degrees
- moved C23 48.6 mm to (6.99, 27.0), turned to 180 degrees
- moved R2 48.0 mm to (56.8, 34.9), turned to 180 degrees
- moved C4 47.3 mm to (54.6, 26.0), turned to 270 degrees
- moved C2 47.2 mm to (56.5, 17.1)
- moved R3 46.7 mm to (56.8, 33.3), turned to 180 degrees
- moved C26 46.0 mm to (10.5, 26.7), flipped to the bottom
- moved R32 45.9 mm to (14.6, 15.2), flipped to the bottom
- moved C6 43.4 mm to (46.4, 32.1), flipped to the bottom, turned to 0 degrees
- moved R33 42.2 mm to (18.4, 34.9), turned to 90 degrees
- moved C5 40.9 mm to (56.5, 26.0), flipped to the top, turned to 270 degrees
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- renumbered BAT2 to BAT1, D4 to D3, IC4 to IC3, JP2 to JP1, LED3 to LED1, TLV320AIC3107 to TLV320AIC1, U10 to U5
Connections:
- net +12V: now also C48.+, R32.1; no longer C51.+, R69.1
- net +3V3: now also C10.1, C11.1, C20.1, C21.1, C22.1, C31.2, C32.2, C33.2, C34.2, C36.2, C43.1, C44.1, C47.2, C57.2, C9.1, R26.2, R27.2, R30.2, R33.2, U1.3, U6.1; no longer C1.1, C16.1, C17.1, C27.1, C28.1, C29.1, C30.1, C39.2, C40.2, C43.2, C45.2, C46.2, C47.1, C5.2, C9.2, R20.2, R47.2, R8.2, R9.2, U4.1, U4.3
- net +5V: now also C18.1, C19.1, C29.1, C30.1, C39.2, C40.2, C7.1, C8.1, L6.2, R37.2, R39.1, U4.5; no longer C11.1, C12.1, C13.1, C14.1, C2.1, C57.2, C6.1, C7.2, L11.2, R70.2, R86.1, U1.5
- net +5V_OTG_PWR: now also C23.1, L3.1; no longer C4.1, L1.1
- net AGND: now also C45.1, C46.1, L5.2; no longer C18.1, C19.1, L2.2
- net DCAN0_RX: now also U2.4; no longer U6.4
- net DCAN0_TX: now also U2.1; no longer U6.1
- net DCAN1_RX: now also U1.4; no longer U2.4
- net DCAN1_TX: now also U1.1; no longer U2.1
- net DVDD: now also C37.2, C59.2, U6.5; no longer C36.2, C44.2, U4.5
- net EXT_WAKEUP: now also R34.1; no longer R54.1
- net GND: now also C18.2, C19.2, C20.2, C21.2, C22.2, C23.2, C24.2, C25.2, C26.2, C31.1, C32.1, C33.1, C34.1, C43.2, C44.2, C47.1, C48.-, C49.2, C50.2, C58.1, C59.1, C7.2, C9.2, L1.1, L5.1, R12.2, R15.1, R16.1, R17.1, R18.1, R31.2, R35.2, R36.2, R41.1; no longer C1.2, C12.2, C13.2, C14.2, C16.2, C2.2, C3.2, C31.2, C32.2, C4.2, C43.1, C44.1, C45.1, C46.1, C47.2, C48.2, C5.1, C51.-, C52.2, C63.2, C64.2, C7.1, C9.1, L3.1, L6.1, R21.1, R24.1, R3.1, R4.1, R41.2, R55.2, R84.2, R85.2
- net GNDA: now also C1.2, C12.2, C13.2, C14.2, C16.2, C17.1, C2.2, C3.2, C4.2, C5.2, C6.1, R1.1, R41.2, R8.1; no longer C20.2, C21.2, C22.2, C23.2, C24.2, C25.2, C26.2, C31.1, C32.1, C33.2, C34.2, R25.1, R26.1
- net HS-CAN_H: now also D1.2, R2.2, R6.2; no longer D2.2, R29.2, R31.2
- net HS-CAN_L: now also D1.1, R7.1; no longer D2.1, R30.1
- net HS-CAN_RS: now also R4.2; no longer R7.2
- net I2C0-SCL: now also R26.1; no longer R8.1
- net I2C0-SDA: now also R27.1; no longer R9.1
- net LED1: now also R38.1; no longer R48.1
- net LED2: now also R40.1; no longer R49.1
- net MS-CAN_H: now also D2.2, R13.1, R9.2; no longer D1.2, R27.1, R6.2
- net MS-CAN_L: now also D2.1, R14.1; no longer D1.1, R28.1
- net MS-CAN_RS: now also R11.2; no longer R40.2
- net N$1: now also R40.2; no longer R49.2
- net N$10: now also C14.1, R10.1, R9.1; no longer C34.1, R33.1, R6.1
- net N$100: now also C25.1, C27.1, L3.2, R20.2, U3.1; no longer C63.1, C64.1, L1.2, R1.2, U1.1
- net N$11: now also C52.2, R35.1; no longer C50.2, R84.1
- net N$12: now also C58.2, U6.4; no longer C37.2, U4.4
- net N$129: now also R39.2; no longer R86.2
- net N$13: now also C26.1, C28.1, L4.1, R23.2, U4.1; no longer C10.1, C8.1, L5.1, R22.2, U3.1
- net N$15: now also C45.2, R29.2; no longer C18.2, R13.2
- net N$16: now also C46.2, R28.2; no longer C19.2, R14.2
- net N$17: now also R28.1; no longer R14.1
- net N$18: now also R29.1; no longer R13.1
- net N$2: now also C3.1, R2.1, R3.1; no longer C33.1, R31.1, R32.1
- net N$231: now also R38.2; no longer R48.2
- net N$266: now also L1.2; no longer L3.2
- net N$27: now also R33.1; no longer R20.1
- net N$28: now also C24.1, L4.2; no longer C3.1, L5.2
- net N$29: now also L2.2; no longer L6.2
- net N$3: now also R16.2, U4.3; no longer R19.2, U3.3
- net N$30: now also R3.2; no longer R32.2
- net N$31: now also C1.1, C2.1, C4.1, C5.1; no longer C23.1, C24.1, C25.1, C26.1
- net N$32: now also R10.2; no longer R33.2
- net N$33: now also R8.2; no longer R25.2
- net N$4: now also C50.1; no longer C52.1
- net N$40: now also R13.2, U2.7; no longer R27.2, U6.7
- net N$41: now also R7.2, U1.6; no longer R30.2, U2.6
- net N$42: now also R14.2, U2.6; no longer R28.2, U6.6
- net N$43: now also R30.1; no longer R47.1
- net N$44: now also C49.1, R31.1, R34.2; no longer C48.1, R54.2, R55.1
- net N$45: now also R6.1, U1.7; no longer R29.1, U2.7
- net N$5: now also R4.1, U1.8; no longer R7.1, U2.8
- net N$50: now also C12.1, C13.1, C16.1; no longer C20.1, C21.1, C22.1
- net N$52: now also R1.2; no longer R26.2
- net N$6: now also R32.2; no longer R69.2
- net N$62: now also R36.1, R37.1; no longer R70.1, R85.1
- net N$7: now also C51.1; no longer C49.1
- net N$8: now also C51.2, L6.1; no longer C49.2, L11.1
- net N$80: now also R11.1, R12.1, U2.8; no longer R40.1, R41.1, U6.8
- net N$9: now also C52.1; no longer C50.1
- net N$99: now also R15.2, U3.3; no longer R3.2, U1.3
- net USB0_CE: now also R21.2; no longer R2.2
- net USB0_DRV: now also R22.2; no longer R34.2
- net USB0_EN: now also R17.2, R21.1, R22.1, U3.4; no longer R2.1, R34.1, R4.2, U1.4
- net USB0_VBUS: now also R20.1; no longer R1.1
- net USB1_CE: now also R24.2; no longer R23.2
- net USB1_DRV: now also R25.2; no longer R35.2
- net USB1_EN: now also R18.2, R24.1, R25.1, U4.4; no longer R21.2, R23.1, R35.1, U3.4
- net USB1_ID: now also R19.2; no longer R24.2
- net USB1_VBUS: now also R23.1; no longer R22.1
Routing:
- net +3V3: track 0.00 -> 16.5 mm
- net N$18: track 0.00 -> 5.91 mm
- net +5V: track 0.00 -> 3.30 mm
- net DVDD: track 0.00 -> 3.12 mm
- net N$17: track 0.00 -> 2.73 mm
