File: interface/Designs/OOBDtiger/ARM_CortexA8_DEBIAN/D5/pcb/OOBD-Tiger.sch (EAGLE design)
At the start: 88 parts, among them IC3 DS1307, IC4 DS3231, Q2 32.768kHz, U1 SY6280, U10 MP1482DS, U2 SN65HVD230(SO8), U6 SN65HVD230(SO8)

Commit message: - delete unneeded nets - connect DCAN0, DCAN1, RTC und Audio to AM3352 GPIO (X-Check necessary) - minor cosmetic stuff
Parts:
- removed JP2: (no value), SparkFun:JUMPER-2SMD-NO
- added R20: 10k, rcl:R-EU_R0603
- R10, R11, R12, R13, R14, R15, R16, R17, R18: device SparkFun-Passives:RESISTOR0805-RES -> resistor:R-EU_R0603
- R8, R9: device SparkFun-Passives:RESISTOR0402-RES -> resistor:R-EU_R0603
- renumbered U$2 to TLV320AIC3107
Connections:
- net P0_12/I2C2_SDA renamed DCAN0_TX
- net P0_13/I2C2_SCL renamed DCAN0_RX
- net P1_8/UART4_RXD renamed DCAN1_TX
- net P1_9/UART4_TXD renamed DCAN1_RX
- net USB1-VBUS renamed USB1_VBUS
- net USB1-VBUS1 renamed USB1_VBUS1
- removed net 3.3V: C16.1, C17.1, R8.2, R9.2, TLV320AIC3107.DRVDD_0, TLV320AIC3107.DRVDD_1, TLV320AIC3107.IOVDD
- removed net AIN4: AM3352-SOM-EVB-PLATFORM.AIN4
- removed net AIN5: AM3352-SOM-EVB-PLATFORM.AIN5
- removed net AIN6: AM3352-SOM-EVB-PLATFORM.AIN6
- removed net AIN7: AM3352-SOM-EVB-PLATFORM.AIN7
- removed net JTAG_TCK: AM3352-SOM-EVB-PLATFORM.JTAG_TCK
- removed net JTAG_TDI: AM3352-SOM-EVB-PLATFORM.JTAG_TDI
- removed net JTAG_TDO: AM3352-SOM-EVB-PLATFORM.JTAG_TDO
- removed net JTAG_TMS: AM3352-SOM-EVB-PLATFORM.JTAG_TMS
- removed net JTAG_TRST: AM3352-SOM-EVB-PLATFORM.JTAG_TRST
- removed net MMC0-SDCD#/EMU4: AM3352-SOM-EVB-PLATFORM.MMC0-SDCD#/EMU4
- removed net N$10: R9.1, TLV320AIC3107.SDA
- removed net NNMI: AM3352-SOM-EVB-PLATFORM.NNMI
- removed net OUT: JP2.2
- removed net P0_0/EMDIO: AM3352-SOM-EVB-PLATFORM.P0_0/EMDIO
- removed net P0_1/EMDC: AM3352-SOM-EVB-PLATFORM.P0_1/EMDC
- removed net P0_14/UART1_RXD: AM3352-SOM-EVB-PLATFORM.P0_14/UART1_RXD
- removed net P0_15/UART1_TXD: AM3352-SOM-EVB-PLATFORM.P0_15/UART1_TXD
- removed net P0_16/ETXD3: AM3352-SOM-EVB-PLATFORM.P0_16/ETXD3
- removed net P0_17/ETXD2: AM3352-SOM-EVB-PLATFORM.P0_17/ETXD2
- removed net P0_2/SPI0_SCLK: AM3352-SOM-EVB-PLATFORM.P0_2/SPI0_SCLK
- removed net P0_20/EMU3: AM3352-SOM-EVB-PLATFORM.P0_20/EMU3
- removed net P0_21/ETXD1: AM3352-SOM-EVB-PLATFORM.P0_21/ETXD1
- removed net P0_28/ETXD0: AM3352-SOM-EVB-PLATFORM.P0_28/ETXD0
- removed net P0_29/EPHY-RST#/RFCLK: AM3352-SOM-EVB-PLATFORM.P0_29/EPHY-RST#/RFCLK
- removed net P0_3/SPI0_D0(MISO): AM3352-SOM-EVB-PLATFORM.P0_3/SPI0_D0(MISO)
- removed net P0_4/SPI0_D1(MOSI): AM3352-SOM-EVB-PLATFORM.P0_4/SPI0_D1(MOSI)
- removed net P0_5/SPI0_CS0: AM3352-SOM-EVB-PLATFORM.P0_5/SPI0_CS0
- removed net P0_7/PWM0_OUT: AM3352-SOM-EVB-PLATFORM.P0_7/PWM0_OUT
- removed net P2_18/ERXD3: AM3352-SOM-EVB-PLATFORM.P2_18/ERXD3
- removed net P2_19/ERXD2: AM3352-SOM-EVB-PLATFORM.P2_19/ERXD2
- removed net P2_20/ERXD1: AM3352-SOM-EVB-PLATFORM.P2_20/ERXD1
- removed net P2_21/ERXD0: AM3352-SOM-EVB-PLATFORM.P2_21/ERXD0
- removed net P3_0/ECOL: AM3352-SOM-EVB-PLATFORM.P3_0/ECOL
- removed net P3_1/ECRS: AM3352-SOM-EVB-PLATFORM.P3_1/ECRS
- removed net P3_10/ERXCK: AM3352-SOM-EVB-PLATFORM.P3_10/ERXCK
- removed net P3_14/SPI1_CLK: AM3352-SOM-EVB-PLATFORM.P3_14/SPI1_CLK
- removed net P3_15/SPI1_D0(MISO): AM3352-SOM-EVB-PLATFORM.P3_15/SPI1_D0(MISO)
- removed net P3_16/SPI1_D1(MOSI): AM3352-SOM-EVB-PLATFORM.P3_16/SPI1_D1(MOSI)
- removed net P3_17/SPI1_CS0: AM3352-SOM-EVB-PLATFORM.P3_17/SPI1_CS0
- removed net P3_18/LED1: AM3352-SOM-EVB-PLATFORM.P3_18/LED1
- removed net P3_2/ERXERR: AM3352-SOM-EVB-PLATFORM.P3_2/ERXERR
- removed net P3_3/ETXEN: AM3352-SOM-EVB-PLATFORM.P3_3/ETXEN
- removed net P3_4/ERXDV: AM3352-SOM-EVB-PLATFORM.P3_4/ERXDV
- removed net P3_5/I2C0-SDA: AM3352-SOM-EVB-PLATFORM.P3_5/I2C0-SDA
- removed net P3_6/I2C0-SCL: AM3352-SOM-EVB-PLATFORM.P3_6/I2C0-SCL
- removed net P3_7/EMU0: AM3352-SOM-EVB-PLATFORM.P3_7/EMU0
- removed net P3_8/EMU1: AM3352-SOM-EVB-PLATFORM.P3_8/EMU1, R40.2, R7.2
- removed net P3_9/ETXCK: AM3352-SOM-EVB-PLATFORM.P3_9/ETXCK
- removed net SCL: IC3.SCL, IC4.SCL, R8.1, TLV320AIC3107.SCL
- removed net SDA: IC3.SDA, IC4.SDA
- removed net V+: C9.2, IC4.VCC, R19.2
- removed net VDDA_ADC: AM3352-SOM-EVB-PLATFORM.VDDA_ADC
- removed net VREFP: AM3352-SOM-EVB-PLATFORM.VREFP
- new net +3V3: C16.1, C17.1, C9.2, IC4.VCC, R20.2, R8.2, R9.2, TLV320AIC3107.DRVDD_0, TLV320AIC3107.DRVDD_1, TLV320AIC3107.IOVDD
- new net HS-CAN_RS: AM3352-SOM-EVB-PLATFORM.P3_8/EMU1, R7.2
- new net I2C0-SCL: AM3352-SOM-EVB-PLATFORM.P3_6/I2C0-SCL, IC3.SCL, IC4.SCL, R8.1, TLV320AIC3107.SCL
- new net I2C0-SDA: AM3352-SOM-EVB-PLATFORM.P3_5/I2C0-SDA, IC3.SDA, IC4.SDA, R9.1, TLV320AIC3107.SDA
- new net MS-CAN_RS: AM3352-SOM-EVB-PLATFORM.P3_7/EMU0, R40.2
- net +5V: now also R19.2
- net AUD_BCLK: now also AM3352-SOM-EVB-PLATFORM.P3_14/SPI1_CLK
- net AUD_DIN: now also AM3352-SOM-EVB-PLATFORM.P3_16/SPI1_D1(MOSI)
- net AUD_DOUT: now also AM3352-SOM-EVB-PLATFORM.P3_17/SPI1_CS0
- net AUD_MCLK: now also AM3352-SOM-EVB-PLATFORM.P3_21/LED3
- net AUD_WCLK: now also AM3352-SOM-EVB-PLATFORM.P3_15/SPI1_D0(MISO)
- net N$27: now also IC4.!INT, R20.1; no longer IC4.!RST
- net N$3: no longer IC4.!INT, JP2.1
- net P3_20/LED2: no longer AM3352-SOM-EVB-PLATFORM.P3_20/LED2
- net P3_21/LED3: no longer AM3352-SOM-EVB-PLATFORM.P3_21/LED3
- net SYS_RESETN: now also IC4.!RST, TLV320AIC3107.RESETN; no longer AM3352-SOM-EVB-PLATFORM.SYS_RESETN@2
Other:
- note removed: "DCAN1_RX"
- note removed: "DCAN1_TX"
- note removed: "LED2"
- note removed: "LED3"
- note removed: "NC (PWRONRSTN)"
- moved on the sheet: BAT1, BAT2, IC3, Q2, R19
