File: interface/Designs/OOBDpiCAN/pcb/sch/OOBDpiCAN.sch (EAGLE design)
At the start: 73 parts, among them Q1 16MHz, X1 RASPI_BOARD_B+_H

Commit message: add USB-HUB GL850G lbr
Parts:
- added U$14: GL850G-31, pimoroni:GL850G-31
Changed lines of the file:
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@@
 <part name="X1" library="raspberrypi_bastelstube_v13" deviceset="RASPI_BOARD_B+" device="_H"/>
 <part name="FRAME3" library="frames" deviceset="A3L-LOC" device=""/>
+<part name="FRAME4" library="frames" deviceset="A3L-LOC" device=""/>
+<part name="U$14" library="pimoroni" deviceset="GL850G-31" device=""/>
 </parts>
 <sheets>
@@
 <instances>
 <instance part="FRAME3" gate="G$1" x="0" y="0"/>
-<instance part="X1" gate="G$1" x="132.08" y="137.16"/>
+<instance part="U$14" gate="G$1" x="180.34" y="144.78"/>
 </instances>
 <busses>
+</busses>
+<nets>
+</nets>
+</sheet>
+<sheet>
+<plain>
+<text x="344.17" y="20.32" size="2.54" layer="94">Author: M. Luxen</text>
+<text x="289.56" y="20.32" size="2.54" layer="94">Title:</text>
+<text x="289.56" y="16.51" size="2.54" layer="94">Raspi 1/2/3 Interface</text>
+</plain>
+<instances>
+<instance part="FRAME4" gate="G$1" x="0" y="0"/>
+<instance part="X1" gate="G$1" x="147.32" y="121.92"/>
+</instances>
+<busses>

Commit message: 4Port USB Hub GL850G connected add ISO1050 alternative CAN interfaces
Parts:
- removed U$13: (no value), SparkFun-Connectors:M03
- removed U$14: GL850G-31, pimoroni:GL850G-31
- added $$U$13: MCP2551SO8, can:MCP2551SO8
- added $$U$14: (no value), SparkFun-Connectors:M03
- added C27, C29, C32, C34, C35, C36, C38, C39, C40, C42, C43, C44, C45, C47, C48, C49, C50, C52: 100nF, resistor:C-EUC0603
- added C28: 22uF/6.3V, rcl:CPOL-EUSMCA
- added C30, C31: 18pF, resistor:C-EUC0603
- added C33: 1uF, resistor:C-EUC0603
- added C37, C41, C46, C51: NA(10nF), resistor:C-EUC0603
- added CN1: (no value), adafruit:USBMOLEX
- added D1, D2, D3, D4: PESD1CAN, Industrialberry:PESD1CAN
- added DC1, DC2, DC3, DC4: (no value), Industrialberry:R1SE
- added IC1, IC2, IC3, IC4: (no value), Industrialberry:ISO1050SO-08
- added L1, L3, L4, L5, L6, L7: 2508056017Y2, rcl:L-EUL0805
- added L2: NA(2508056017Y2), rcl:L-EUL0805
- added Q2: 16MHz, crystal:CRYSTALSM49
- added R17: NA(47k), resistor:R-EU_R0603
- added R18: 680R, resistor:R-EU_R0603
- added R19: 10k, resistor:R-EU_R0603
- added R20, R21, R22, R23, R24, R25, R26: 60R, resistor:R-EU_R0603
- C1, C2: value 100nF -> 33pF
- C11, C12, C14: value 18pF -> 100nF
- C9: value 100nF -> 22uF/6.3V; device resistor:C-EUC0603 -> rcl:CPOL-EUSMCA
- LED2, LED4: value green -> yellow
- LED5, LED7: value yellow -> green
- Q1: value 16MHz -> 12MHz
- R1, R2: value 510R -> 10k
- R11, R3, R4: value 120R -> 510R
- R16: value 120R -> 10k
- R9: value 510R -> 60R
- U$1, U$9: value STM32F042CT -> MCP2551SO8; device micro-stm_v3:STM32F042CT -> can:MCP2551SO8
- U$10: value MCP2551SO8 -> (none); device can:MCP2551SO8 -> SparkFun-Connectors:M03
- U$3: value MCP2551SO8 -> GL850G-31; device can:MCP2551SO8 -> pimoroni:GL850G-31
- U$4: value MCP2551SO8 -> STM32F042CT; device can:MCP2551SO8 -> micro-stm_v3:STM32F042CT
- U$5: value (none) -> STM32F042CT; device SparkFun-Connectors:M03 -> micro-stm_v3:STM32F042CT
- U$6: value (none) -> STM32F042CT; device jumper:JP5E -> micro-stm_v3:STM32F042CT
- U$8: value STM32F042CT -> (none); device micro-stm_v3:STM32F042CT -> jumper:JP5E
Connections:
- net MC0_2 renamed MCO_0
- removed net N$1: U$10G$1.RXD, U$8.PB8
- removed net N$5: U$10G$1.TXD, U$8.PB9
- removed net N$9 (its old number): LED6.C, R12.2
- removed net NRST3: U$2.NRST
- removed net SWCLK2: U$1.PA14, U$6.2
- removed net SWCLK3: U$2.PA14
- removed net SWDIO2: U$1.PA13, U$6.4
- removed net SWDIO3: U$2.PA13
- removed net USB0_DM1: U$9.PA11
- removed net USB0_DM2: U$1.PA11
- removed net USB0_DM3: U$2.PA11
- removed net USB0_DP1: U$9.PA12
- removed net USB0_DP2: U$1.PA12
- removed net USB0_DP3: U$2.PA12
- new net CAN1-H: D1.C2, IC1.CANH, R20.1, U$1G$1.CANH, U$7.3
- new net CAN1-L: D1.C1, IC1.CANL, JP3.2, U$1G$1.CANL, U$7.2
- new net CAN2-H: D3.C2, IC3.CANH, R23.1, U$11G$1.CANH, U$12.3
- new net CAN2-L: D3.C1, IC3.CANL, JP7.2, U$11G$1.CANL, U$12.2
- new net CAN3-H: $$U$13G$1.CANH, $$U$14.3, D4.C2, IC4.CANH, R25.1
- new net CAN3-L: $$U$13G$1.CANL, $$U$14.2, D4.C1, IC4.CANL, JP8.2
- new net N$17: LED4.C, R14.2
- new net N$2: C1.1, Q1.2, U$3.X2
- new net N$3: C2.1, Q1.1, U$3.X1
- new net N$33: C6.1, C9.+, L1.2, R1.2, R2.2, U$3.DVDD, U$3.V33
- new net N$34: R2.1, U$3.PGANG
- new net N$35: R1.1, U$3.PSELF
- new net N$36: C33.1, R16.2, R17.2, U$3.RESET#
- new net N$37: CN1.D+, U$3.DP0
- new net N$38: CN1.D-, U$3.DM0
- new net N$39: C3.1, C4.1, C5.1, L1.1, U$3.AVDD, U$3.AVDD2, U$3.AVDD3
- new net N$40: R18.2, U$3.RREF
- new net N$41: CN1.GND, L3.2
- new net N$42: CN1.VBUS, L2.2
- new net N$43: C34.1, DC1.VIN+, L4.2
- new net N$44: CN1.ID, R19.2
- new net N$45: C35.1, C35.2, DC1.VOUT+, IC1.VCC2
- new net N$46: IC2.TXD, U$2.PB9, U$9G$1.TXD
- new net N$47: DC1.VOUT-, IC1.GND2
- new net N$48: JP6.1, R22.1
- new net N$49: C37.1, R20.2, R9.2
- new net N$50: C39.1, DC2.VIN+, L5.2
- new net N$51: C38.1, C38.2, DC2.VOUT+, IC2.VCC2
- new net N$52: DC2.VOUT-, IC2.GND2
- new net N$53: C41.1, R21.2, R22.2
- new net N$54: $$U$13G$1.TXD, IC4.TXD, U$6.PB9
- new net N$56: IC3.RXD, U$11G$1.RXD, U$5.PB8
- new net N$57: IC3.TXD, U$11G$1.TXD, U$5.PB9
- new net N$59: JP8.1, R26.1
- new net N$60: C49.1, DC4.VIN+, L7.2
- new net N$61: C48.1, C48.2, DC4.VOUT+, IC4.VCC2
- new net N$62: DC4.VOUT-, IC4.GND2
- new net N$63: C51.1, R25.2, R26.2
- new net USB1_DM: U$3.DM2, U$4.PA11
- new net USB1_DP: U$3.DP2, U$4.PA12
- new net USB2_DM: U$3.DM3, U$5.PA11
- new net USB2_DP: U$3.DP3, U$5.PA12
- new net USB3_DM: U$3.DM4, U$6.PA11
- new net USB3_DP: U$3.DP4, U$6.PA12
- net +3V3: now also C11.1, C12.1, C13.1, C14.1, C25.1, C26.1, C27.1, C29.1, JP4.1, U$4.VBAT, U$4.VDD1, U$4.VDD2, U$4.VDDA, U$4.VDDIO2, U$5.VBAT, U$5.VDD1, U$5.VDD2, U$5.VDDA, U$5.VDDIO2, U$6.VBAT, U$6.VDD1, U$6.VDD2, U$6.VDDA, U$6.VDDIO2, U$8.1; no longer C1.1, C18.1, C2.1, C3.1, C4.1, C5.1, C6.1, C9.1, JP6.1, U$1.VBAT, U$1.VDD1, U$1.VDD2, U$1.VDDA, U$1.VDDIO2, U$6.1, U$8.VBAT, U$8.VDD1, U$8.VDD2, U$8.VDDA, U$8.VDDIO2, U$9.VBAT, U$9.VDD1, U$9.VDD2, U$9.VDDA, U$9.VDDIO2
- net +5V: now also $$U$13G$2.VCC, C18.1, C28.+, C32.1, C36.1, C40.1, C42.1, C45.1, C47.1, C50.1, C52.1, IC1.VCC1, IC2.VCC1, IC3.VCC1, IC4.VCC1, L2.1, L4.1, L5.1, L6.1, L7.1, R16.1, U$1G$2.VCC, U$3.V5, U$9G$2.VCC; no longer C13.1, C14.1, C25.1, C26.1, U$10G$2.VCC, U$3G$2.VCC, U$4G$2.VCC
- net BOOT0: now also JP4.2, R11.2, R3.2, R4.2, U$4.PF11-BOOT0, U$5.PF11-BOOT0, U$6.PF11-BOOT0; no longer JP6.2, R1.2, R2.2, R9.2, U$1.PF11-BOOT0, U$8.PF11-BOOT0, U$9.PF11-BOOT0
- net CAN0-H: now also D2.C2, IC2.CANH, R21.1, U$10.3, U$9G$1.CANH; no longer R15.2, R16.2, R7.2, R8.2, U$10G$1.CANH, U$11G$1.CANH, U$12.3, U$13.3, U$3G$1.CANH, U$4G$1.CANH, U$5.3, U$7.3
- net CAN0-L: now also D2.C1, IC2.CANL, JP6.2, U$10.2, U$9G$1.CANL; no longer JP3.2, JP4.2, JP7.2, JP8.2, U$10G$1.CANL, U$11G$1.CANL, U$12.2, U$13.2, U$3G$1.CANL, U$4G$1.CANL, U$5.2, U$7.2
- net GND: now also $$U$13G$1.RS, $$U$13G$2.GND, $$U$14.4, C27.2, C28.-, C29.2, C30.2, C31.2, C32.2, C33.2, C34.2, C36.2, C37.2, C39.2, C40.2, C41.2, C42.2, C44.2, C45.2, C46.2, C47.2, C49.2, C50.2, C51.2, C52.2, C9.-, D1.CC, D2.CC, D3.CC, D4.CC, DC1.VIN-, DC2.VIN-, DC3.VIN-, DC4.VIN-, IC1.GND1, IC2.GND1, IC3.GND1, IC4.GND1, L3.1, R15.1, R17.1, R18.1, R19.1, R7.1, R8.1, U$10.4, U$1G$1.RS, U$1G$2.GND, U$3.GND, U$3.TEST/SCL, U$4.VSS1, U$4.VSS2, U$4.VSS3, U$4.VSSA, U$5.VSS1, U$5.VSS2, U$5.VSS3, U$5.VSSA, U$6.VSS1, U$6.VSS2, U$6.VSS3, U$6.VSSA, U$8.3, U$9G$1.RS, U$9G$2.GND; no longer C9.2, R1.1, R2.1, R9.1, U$1.VSS1, U$1.VSS2, U$1.VSS3, U$1.VSSA, U$10G$1.RS, U$10G$2.GND, U$13.4, U$3G$1.RS, U$3G$2.GND, U$4G$1.RS, U$4G$2.GND, U$5.4, U$6.3, U$8.VSS1, U$8.VSS2, U$8.VSS3, U$8.VSSA, U$9.VSS1, U$9.VSS2, U$9.VSS3, U$9.VSSA
- net MC0_1: now also U$4.PA8, U$5.PF0-OSC_IN; no longer U$8.PF0-OSC_IN
- net MCO_1: now also U$4.PF0-OSC_IN; no longer U$1.PA8, U$2.PF0-OSC_IN
- net MCO_2: now also U$5.PA8, U$6.PF0-OSC_IN; no longer U$8.PA8, U$9.PF0-OSC_IN
- net N$10: now also C31.1, Q2.2, U$2.PF1-OSC_OUT; no longer C12.1, Q1.2, U$1.PF1-OSC_OUT
- net N$11: now also C30.1, Q2.1, U$2.PF0-OSC_IN; no longer C11.1, Q1.1, U$1.PF0-OSC_IN
- net N$12: now also C44.1, DC3.VIN+, L6.2; no longer U$11G$1.RXD, U$9.PB8
- net N$13: now also C43.1, C43.2, DC3.VOUT+, IC3.VCC2; no longer U$11G$1.TXD, U$9.PB9
- net N$14: now also DC3.VOUT-, IC3.GND2; no longer JP8.1, R16.1
- net N$15: now also LED4.A, U$6.PB1; no longer LED7.A, U$9.PB1
- net N$16: now also U$6.PB0; no longer U$9.PB0
- net N$18: now also R15.2; no longer R14.2
- net N$19: now also IC2.RXD, U$2.PB8, U$9G$1.RXD; no longer U$1.PB8, U$3G$1.RXD
- net N$20: now also C46.1, R23.2, R24.2; no longer U$1.PB9, U$3G$1.TXD
- net N$21: now also $$U$13G$1.RXD, IC4.RXD, U$6.PB8; no longer JP3.1, R7.1
- net N$22: now also U$2.PB1; no longer U$1.PB1
- net N$23: now also LED5.A, U$2.PB0; no longer LED2.A, U$1.PB0
- net N$24: now also R5.2; no longer R3.2
- net N$25: now also LED5.C, R6.2; no longer LED2.C, R4.2
- net N$26: now also IC1.RXD, U$1G$1.RXD, U$4.PB8; no longer U$2.PB8, U$4G$1.RXD
- net N$27: now also IC1.TXD, U$1G$1.TXD, U$4.PB9; no longer U$2.PB9, U$4G$1.TXD
- net N$28: now also JP3.1, R9.1; no longer JP4.1, R8.1
- net N$29: now also LED2.A, U$4.PB1; no longer LED3.A, U$2.PB1
- net N$30: now also LED6.A, U$4.PB0; no longer LED4.A, U$2.PB0
- net N$31: now also LED2.C, R7.2; no longer LED3.C, R5.2
- net N$32: now also LED6.C, R8.2; no longer LED4.C, R6.2
- net N$4: now also LED3.A, U$5.PB1; no longer LED5.A, U$8.PB1
- net N$6: now also R24.1; no longer R15.1
- net N$7: now also LED7.A, U$5.PB0; no longer LED6.A, U$8.PB0
- net N$8: now also LED3.C, R12.2; no longer LED5.C, R11.2
- net NRST: now also U$4.NRST, U$5.NRST, U$8.5; no longer U$8.NRST
- net NRST1: now also U$6.NRST; no longer U$9.NRST
- net NRST2: now also U$2.NRST; no longer U$1.NRST, U$6.5
- net SWCLK: now also U$2.PA14, U$4.PA14, U$5.PA14, U$8.2; no longer U$8.PA14
- net SWCLK1: now also U$6.PA14; no longer U$9.PA14
- net SWDIO: now also U$2.PA13, U$4.PA13, U$5.PA13, U$8.4; no longer U$8.PA13
- net SWDIO1: now also U$6.PA13; no longer U$9.PA13
- net USB0_DM: now also U$2.PA11, U$3.DM1; no longer U$8.PA11
- net USB0_DP: now also U$2.PA12, U$3.DP1; no longer U$8.PA12

Commit message: - fix ERC (Pwr supply) issues due to faulty GL850G symbol - exchange ISO1050 against ADMU3053 and limit to a max of 2x galvanic isolated CAN-Interface due to size of PCB
Parts:
- removed C47, C48, C49, C52: 100nF, resistor:C-EUC0603
- removed DC1, DC2, DC3, DC4: (no value), Industrialberry:R1SE
- removed IC2, IC3, IC4: (no value), Industrialberry:ISO1050SO-08
- removed L4, L5, L6, L7: 2508056017Y2, rcl:L-EUL0805
- removed X1: RASPI_BOARD_B+_H, raspberrypi_bastelstube_v13:RASPI_BOARD_B+_H
- added BAT2: (no value), SparkFun:BATTERY12PTH
- added C53: 1uF, rcl:C-EUC0603
- added C54: 100nF, rcl:C-EUC0603
- added C55: 10n, rcl:C-EUC0603K
- added C56, C58: 100n, rcl:C-EUC0603K
- added C57, C61: 10u, rcl:C-EUC0805K
- added C59, C62: 100n, rcl:C-EUC0805K
- added C60: 10n, rcl:C-EUC0805K
- added IC5: DS3231, DS3231_industrialberry:DS3231SOIC-16W
- added IC6: EEPROM24, FLYFISH:EEPROM24
- added IC7: ADM3053M, ADM3053:ADM3053M
- added JP10: (no value), SparkFun:JUMPER-2SMD-NO
- added JP9: (no value), MirkoSmartSpaceSolutions:MA03-1
- added R27, R28, R29, R30: 10k, rcl:R-EU_R0603
- added R31, R32: 8.2k, rcl:R-EU_R0603
- added R33: (no value), rcl:R-EU_0204/7
- added RPI1: (no value), Connector_B+:RASPBERRY_HATHAT
- added SJ2: SOLDERJUMPERTRACE, SparkFun:SOLDERJUMPERTRACE
- C34: value 100nF -> 10n; device resistor:C-EUC0603 -> rcl:C-EUC0603K
- C35, C38: value 100nF -> 100n; device resistor:C-EUC0603 -> rcl:C-EUC0603K
- C36, C43: value 100nF -> 10u; device resistor:C-EUC0603 -> rcl:C-EUC0805K
- C39, C44: value 100nF -> 100n; device resistor:C-EUC0603 -> rcl:C-EUC0805K
- C42: value 100nF -> 10n; device resistor:C-EUC0603 -> rcl:C-EUC0805K
- C46: value NA(10nF) -> NA(47nF)
- IC1: value (none) -> ADM3053M; device Industrialberry:ISO1050SO-08 -> ADM3053:ADM3053M
Connections:
- net N$26 renamed CAN1_RXD
- net N$27 renamed CAN1_TXD
- removed net N$14: DC3.VOUT-, IC3.GND2
- removed net N$19: IC2.RXD, U$2.PB8, U$9G$1.RXD
- removed net N$43: C34.1, DC1.VIN+, L4.2
- removed net N$45: C35.1, C35.2, DC1.VOUT+, IC1.VCC2
- removed net N$46: IC2.TXD, U$2.PB9, U$9G$1.TXD
- removed net N$47: DC1.VOUT-, IC1.GND2
- removed net N$50: C39.1, DC2.VIN+, L5.2
- removed net N$51: C38.1, C38.2, DC2.VOUT+, IC2.VCC2
- removed net N$52: DC2.VOUT-, IC2.GND2
- removed net N$60: C49.1, DC4.VIN+, L7.2
- removed net N$61: C48.1, C48.2, DC4.VOUT+, IC4.VCC2
- removed net N$62: DC4.VOUT-, IC4.GND2
- new net CAN0_RXD: IC7.RXD, U$2.PB8, U$9G$1.RXD
- new net CAN0_TXD: IC7.TXD, U$2.PB9, U$9G$1.TXD
- new net GNDA: C39.2, C42.2, C43.2, C44.2, C59.2, C60.2, C61.2, C62.2, IC1.GND2@0, IC1.GND2@1, IC1.GND2@2, IC1.GND2@3, IC7.GND2@0, IC7.GND2@1, IC7.GND2@2, IC7.GND2@3, R31.1, R32.1
- new net GPIO17: RPI1.GPIO17
- new net ID_SC: IC6.SCL, R28.2, RPI1.ID_SC
- new net ID_SD: IC6.SDA, R29.2, RPI1.ID_SD
- new net INT-: IC5.!INT, JP10.2, R27.1
- new net N$1: IC7.R_S, R31.2
- new net N$5: IC6.WP, R30.2, SJ2.2
- new net N$55: JP10.1
- new net N$65: C59.1, C60.1, C61.1, C62.1, IC7.V_ISOIN, IC7.V_ISOOUT
- new net RXD: JP9.2, RPI1.RXD
- new net SCL: IC5.SCL, RPI1.SCL
- new net SDA: IC5.SDA, RPI1.SDA
- new net TXD: JP9.3, RPI1.TXD
- new net VBAT: BAT2.+, IC5.VBAT
- net +3V3: now also C34.1, C35.1, C53.2, C55.1, C56.1, IC1.V_IO, IC5.VCC, IC7.V_IO, R27.2, RPI1.3V3A, RPI1.3V3B
- net +5V: now also C38.1, C54.2, C57.1, C58.1, IC1.VCC, IC6.VCC, IC7.VCC, R28.1, R29.1, R30.1, RPI1.5V0A, RPI1.5V0B; no longer C42.1, C47.1, C52.1, IC1.VCC1, IC2.VCC1, IC3.VCC1, IC4.VCC1, L4.1, L5.1, L6.1, L7.1
- net CAN0-H: now also IC7.CAN_H; no longer IC2.CANH
- net CAN0-L: now also IC7.CAN_L; no longer IC2.CANL
- net CAN1-H: now also IC1.CAN_H; no longer IC1.CANH
- net CAN1-L: now also IC1.CAN_L; no longer IC1.CANL
- net CAN2-H: no longer IC3.CANH
- net CAN2-L: no longer IC3.CANL
- net CAN3-H: no longer IC4.CANH
- net CAN3-L: no longer IC4.CANL
- net GND: now also BAT2.-, C35.2, C38.2, C53.1, C54.1, C55.2, C56.2, C57.2, C58.2, IC1.GND1@0, IC1.GND1@1, IC1.GND1@2, IC1.GND1@3, IC1.GND1@4, IC5.GND, IC5.NC@1, IC5.NC@2, IC5.NC@3, IC5.NC@4, IC5.NC@5, IC5.NC@6, IC5.NC@7, IC5.NC@8, IC6.A0, IC6.A1, IC6.A2, IC6.GND, IC7.GND1@0, IC7.GND1@1, IC7.GND1@2, IC7.GND1@3, IC7.GND1@4, JP9.1, RPI1.GND_A, RPI1.GND_B, RPI1.GND_C, RPI1.GND_D, RPI1.GND_E, RPI1.GND_F, RPI1.GND_G, RPI1.GND_H, SJ2.1; no longer C39.2, C42.2, C44.2, C47.2, C49.2, C52.2, DC1.VIN-, DC2.VIN-, DC3.VIN-, DC4.VIN-, IC1.GND1, IC2.GND1, IC3.GND1, IC4.GND1
- net N$12: now also IC1.R_S, R32.2; no longer C44.1, DC3.VIN+, L6.2
- net N$13: now also C39.1, C42.1, C44.1, IC1.V_ISOIN, IC1.V_ISOOUT; no longer C43.2, DC3.VOUT+, IC3.VCC2
- net N$21: no longer IC4.RXD
- net N$54: no longer IC4.TXD
- net N$56: no longer IC3.RXD
- net N$57: no longer IC3.TXD
Other:
- note added: "4-Port USB-HUB"
- note added: "EEPROM"
- note added: "Raspi B+ GPIO"
- note added: "Real Time Clock"
- note removed: "Raspi 1/2/3 Interface"

Commit message: exchange X-references from supply2 library to X-Ref symbols
Connections:
- removed net N$55: JP10.1
- removed net NRST2: U$2.NRST
- net GPIO17: now also JP10.1
- net NRST: now also U$2.NRST
Other:
- moved on the sheet: BAT2

Commit message: start placing parts
Parts:
- added R34, R35, R36: 0R, rcl:R-EU_0207/10
- R33: value (none) -> 0R; device rcl:R-EU_0204/7 -> rcl:R-EU_0207/10
Connections:
- new net N$14: R33.1, U$9G$1.CANL
- new net N$19: R34.1, U$9G$1.CANH
- new net N$26: R36.1, U$1G$1.CANH
- new net N$27: R35.1, U$1G$1.CANL
- net CAN0-H: now also R34.2; no longer U$9G$1.CANH
- net CAN0-L: now also R33.2; no longer U$9G$1.CANL
- net CAN1-H: now also R36.2; no longer U$1G$1.CANH
- net CAN1-L: now also R35.2; no longer U$1G$1.CANL
Other:
- note added: "CAN-Interface #1"
- note added: "CAN-Interface #1 and #2"
- note added: "CAN-Interface #2"
- note added: "CAN-Interface #3"
- note added: "CAN-Interface #4"
- moved on the sheet: R33, U$1G$1, U$9G$1

Commit message: first roughly placing of ADM3053
Parts:
- removed C61: 10u, rcl:C-EUC0805K
- removed C62: 100n, rcl:C-EUC0805K
- removed U$10, U$12, U$7: (no value), SparkFun-Connectors:M03
- removed U$8: (no value), jumper:JP5E
- added C47: NA(47nF), resistor:C-EUC0603
- added C48: NA(10nF), resistor:C-EUC0603
- added C49: 33pF, resistor:C-EUC0603
- added C52: 100nF, resistor:C-EUC0603
- added IC11: EEPROM24, FLYFISH:EEPROM24
- added IC12: DS3231, DS3231_industrialberry:DS3231SOIC-16W
- added IC2: STM32F042CT, micro-stm_v3:STM32F042CT
- added IC4: MCP2551SO8, can:MCP2551SO8
- C1, C2: value 33pF -> 100nF
- C11, C12: value 100nF -> 18pF
- C13, C14, C19, C20: value 100nF -> 100n; device resistor:C-EUC0603 -> rcl:C-EUC0603K
- C15, C16, C27, C29: value 100nF -> 10u; device resistor:C-EUC0603 -> rcl:C-EUC0805K
- C17, C18: value 100nF -> 10n; device resistor:C-EUC0603 -> rcl:C-EUC0603K
- C23, C24: value 100nF -> NA (AY2221K29Y5SS63L7); device resistor:C-EUC0603 -> rcl:C-EU075-032X103
- C25, C26: value 100nF -> 100n; device resistor:C-EUC0603 -> rcl:C-EUC0805K
- C28: value 22uF/6.3V -> NA(10nF); device rcl:CPOL-EUSMCA -> resistor:C-EUC0603
- C30: value 18pF -> NA(10nF)
- C31: value 18pF -> 10n; device resistor:C-EUC0603 -> rcl:C-EUC0805K
- C32: value 100nF -> 10n; device resistor:C-EUC0603 -> rcl:C-EUC0805K
- C33: value 1uF -> 100n; device resistor:C-EUC0603 -> rcl:C-EUC0805K
- C34: value 10n -> 100n; device rcl:C-EUC0603K -> rcl:C-EUC0805K
- C35, C38: value 100n -> 100nF; device rcl:C-EUC0603K -> resistor:C-EUC0603
- C36, C43, C57: value 10u -> 100nF; device rcl:C-EUC0805K -> resistor:C-EUC0603
- C37, C41: value NA(10nF) -> 100nF
- C39, C44, C59: value 100n -> 100nF; device rcl:C-EUC0805K -> resistor:C-EUC0603
- C42: value 10n -> 100nF; device rcl:C-EUC0805K -> resistor:C-EUC0603
- C46: value NA(47nF) -> 100nF
- C50: device resistor:C-EUC0603 -> rcl:C-EUC0603
- C51: value NA(10nF) -> 33pF
- C53: value 1uF -> 100nF; device rcl:C-EUC0603 -> resistor:C-EUC0603
- C54: device rcl:C-EUC0603 -> resistor:C-EUC0603
- C55: value 10n -> 1uF; device rcl:C-EUC0603K -> resistor:C-EUC0603
- C56: value 100n -> 1uF; device rcl:C-EUC0603K -> rcl:C-EUC0603
- C58: value 100n -> 22uF/6.3V; device rcl:C-EUC0603K -> rcl:CPOL-EUSMCA
- C60: value 10n -> 22uF/6.3V; device rcl:C-EUC0805K -> rcl:CPOL-EUSMCA
- C9: value 22uF/6.3V -> 100nF; device rcl:CPOL-EUSMCA -> resistor:C-EUC0603
- IC1, IC7: value ADM3053M -> STM32F042CT; device ADM3053:ADM3053M -> micro-stm_v3:STM32F042CT
- IC5: value DS3231 -> ADM3053M; device DS3231_industrialberry:DS3231SOIC-16W -> ADM3053:ADM3053M
- IC6: value EEPROM24 -> ADM3053M; device FLYFISH:EEPROM24 -> ADM3053:ADM3053M
- LED2, LED4: value yellow -> green
- LED5, LED7: value green -> yellow
- Q1: value 12MHz -> 16MHz
- Q2: value 16MHz -> 12MHz
- R1, R2: value 10k -> 510R
- R10: value 510R -> 0R; device resistor:R-EU_R0603 -> rcl:R-EU_0207/10
- R11: value 510R -> 8.2k; device resistor:R-EU_R0603 -> rcl:R-EU_R0603
- R12: value 120R -> 8.2k; device resistor:R-EU_R0603 -> rcl:R-EU_R0603
- R13, R14, R15: value 120R -> 60R
- R16: value 10k -> 60R
- R17: value NA(47k) -> 510R
- R18: value 680R -> 510R
- R19: value 10k -> 120R
- R20, R21, R22: value 60R -> 120R
- R27: value 10k -> 680R; device rcl:R-EU_R0603 -> resistor:R-EU_R0603
- R3, R4: value 510R -> 120R
- R31: value 8.2k -> 10k; device rcl:R-EU_R0603 -> resistor:R-EU_R0603
- R32: value 8.2k -> NA(47k); device rcl:R-EU_R0603 -> resistor:R-EU_R0603
- R33, R34, R36: value 0R -> 10k; device rcl:R-EU_0207/10 -> resistor:R-EU_R0603
- R35: value 0R -> 10k; device rcl:R-EU_0207/10 -> rcl:R-EU_R0603
- R7, R8: value 120R -> 0R; device resistor:R-EU_R0603 -> rcl:R-EU_0207/10
- R9: value 60R -> 0R; device resistor:R-EU_R0603 -> rcl:R-EU_0207/10
- U$1: value MCP2551SO8 -> (none); device can:MCP2551SO8 -> jumper:JP5E
- U$2, U$4: value STM32F042CT -> (none); device micro-stm_v3:STM32F042CT -> SparkFun-Connectors:M03
- U$3: value GL850G-31 -> (none); device pimoroni:GL850G-31 -> SparkFun-Connectors:M03
- U$5: value STM32F042CT -> GL850G-31; device micro-stm_v3:STM32F042CT -> pimoroni:GL850G-31
- renumbered $$U$13 to IC10, $$U$14 to $$U$1, BAT2 to BAT1, SJ2 to SJ1, U$11 to IC9, U$6 to IC8, U$9 to IC3
Connections:
- net +3V3: now also C1.1, C18.1, C2.1, C3.1, C36.1, C37.1, C38.1, C39.1, C4.1, C40.1, C41.1, C42.1, C43.1, C44.1, C5.1, C56.2, C6.1, C9.1, IC1.VBAT, IC1.VDD1, IC1.VDD2, IC1.VDDA, IC1.VDDIO2, IC12.VCC, IC2.VBAT, IC2.VDD1, IC2.VDD2, IC2.VDDA, IC2.VDDIO2, IC5.V_IO, IC6.V_IO, IC7.VBAT, IC7.VDD1, IC7.VDD2, IC7.VDDA, IC7.VDDIO2, JP6.1, R35.2, U$1.1; no longer C11.1, C12.1, C13.1, C14.1, C15.1, C16.1, C21.1, C22.1, C23.1, C24.1, C25.1, C26.1, C27.1, C29.1, C34.1, C53.2, C55.1, C56.1, IC1.V_IO, IC5.VCC, IC7.V_IO, JP4.1, R27.2, U$2.VBAT, U$2.VDD1, U$2.VDD2, U$2.VDDA, U$2.VDDIO2, U$4.VBAT, U$4.VDD1, U$4.VDD2, U$4.VDDA, U$4.VDDIO2, U$5.VBAT, U$5.VDD1, U$5.VDD2, U$5.VDDA, U$5.VDDIO2, U$8.1
- net +5V: now also C13.1, C14.1, C15.1, C16.1, C21.1, C22.1, C46.1, C50.2, C59.1, C60.+, IC11.VCC, IC4G$2.VCC, IC5.VCC, R31.1, U$5.V5; no longer C18.1, C28.+, C32.1, C36.1, C38.1, C40.1, C50.1, C54.2, C57.1, C58.1, IC1.VCC, IC7.VCC, R16.1, U$1G$2.VCC, U$3.V5
- net BOOT0: now also IC1.PF11-BOOT0, IC2.PF11-BOOT0, IC7.PF11-BOOT0, JP6.2, R1.2, R17.2, R18.2, R2.2; no longer JP4.2, R10.2, R11.2, R3.2, R4.2, U$2.PF11-BOOT0, U$4.PF11-BOOT0, U$5.PF11-BOOT0
- net CAN0-H: now also IC5.CAN_H, R14.1, R8.2, U$2.3; no longer IC7.CAN_H, R21.1, R34.2, U$10.3
- net CAN0-L: now also IC5.CAN_L, JP3.2, R7.2, U$2.2; no longer IC7.CAN_L, JP6.2, R33.2, U$10.2
- net CAN0_RXD: now also IC1.PB8, IC5.RXD; no longer IC7.RXD, U$2.PB8
- net CAN0_TXD: now also IC1.PB9, IC5.TXD; no longer IC7.TXD, U$2.PB9
- net CAN1-H: now also IC6.CAN_H, R10.2, R16.1, U$3.3; no longer IC1.CAN_H, R20.1, R36.2, U$7.3
- net CAN1-L: now also IC6.CAN_L, JP4.2, R9.2, U$3.2; no longer IC1.CAN_L, JP3.2, R35.2, U$7.2
- net CAN1_RXD: now also IC2.PB8, IC4G$1.RXD, IC6.RXD; no longer IC1.RXD, U$1G$1.RXD, U$4.PB8
- net CAN1_TXD: now also IC2.PB9, IC4G$1.TXD, IC6.TXD; no longer IC1.TXD, U$1G$1.TXD, U$4.PB9
- net CAN2-H: now also R24.1, U$4.3; no longer R23.1, U$12.3
- net CAN2-L: now also U$4.2; no longer U$12.2
- net CAN3-H: now also R26.1; no longer R25.1
- net GND: now also C23.1, C24.1, C28.2, C39.2, C42.2, C43.2, C44.2, C47.2, C48.2, C49.2, C50.1, C52.2, C53.2, C54.2, C56.1, C58.-, C59.2, C60.-, C9.2, IC1.VSS1, IC1.VSS2, IC1.VSS3, IC1.VSSA, IC11.A0, IC11.A1, IC11.A2, IC11.GND, IC12.GND, IC12.NC@1, IC12.NC@2, IC12.NC@3, IC12.NC@4, IC12.NC@5, IC12.NC@6, IC12.NC@7, IC12.NC@8, IC2.VSS1, IC2.VSS2, IC2.VSS3, IC2.VSSA, IC4G$1.RS, IC4G$2.GND, IC5.GND1@0, IC5.GND1@1, IC5.GND1@2, IC5.GND1@3, IC5.GND1@4, IC6.GND1@0, IC6.GND1@1, IC6.GND1@2, IC6.GND1@3, IC6.GND1@4, IC7.VSS1, IC7.VSS2, IC7.VSS3, IC7.VSSA, R1.1, R2.1, R20.1, R21.1, R22.1, R27.1, R32.1, R36.1, U$1.3, U$2.4, U$3.4, U$4.4, U$5.GND, U$5.TEST/SCL; no longer C23.2, C24.2, C25.2, C26.2, C27.2, C28.-, C29.2, C31.2, C32.2, C33.2, C34.2, C50.2, C53.1, C54.1, C56.2, C58.2, C9.-, IC1.GND1@0, IC1.GND1@1, IC1.GND1@2, IC1.GND1@3, IC1.GND1@4, IC5.GND, IC5.NC@1, IC5.NC@2, IC5.NC@3, IC5.NC@4, IC5.NC@5, IC5.NC@6, IC5.NC@7, IC5.NC@8, IC6.A0, IC6.A1, IC6.A2, IC6.GND, IC7.GND1@0, IC7.GND1@1, IC7.GND1@2, IC7.GND1@3, IC7.GND1@4, R10.1, R11.1, R12.1, R13.1, R14.1, R15.1, R7.1, R8.1, U$10.4, U$12.4, U$1G$1.RS, U$1G$2.GND, U$2.VSS1, U$2.VSS2, U$2.VSS3, U$2.VSSA, U$3.GND, U$3.TEST/SCL, U$4.VSS1, U$4.VSS2, U$4.VSS3, U$4.VSSA, U$5.VSS1, U$5.VSS2, U$5.VSS3, U$5.VSSA, U$7.4, U$8.3
- net GNDA: now also C23.2, C24.2, C25.2, C26.2, C27.2, C29.2, C31.2, C32.2, C33.2, C34.2, IC5.GND2@0, IC5.GND2@1, IC5.GND2@2, IC5.GND2@3, IC6.GND2@0, IC6.GND2@1, IC6.GND2@2, IC6.GND2@3, R11.1, R12.1; no longer C39.2, C42.2, C43.2, C44.2, C59.2, C60.2, C61.2, C62.2, IC1.GND2@0, IC1.GND2@1, IC1.GND2@2, IC1.GND2@3, IC7.GND2@0, IC7.GND2@1, IC7.GND2@2, IC7.GND2@3, R31.1, R32.1
- net ID_SC: now also IC11.SCL, R29.2; no longer IC6.SCL, R28.2
- net ID_SD: now also IC11.SDA, R30.2; no longer IC6.SDA, R29.2
- net INT-: now also IC12.!INT, R35.1; no longer IC5.!INT, R27.1
- net MC0_1: now also IC2.PA8, IC7.PF0-OSC_IN; no longer U$4.PA8, U$5.PF0-OSC_IN
- net MCO_0: now also IC1.PA8; no longer U$2.PA8
- net MCO_1: now also IC2.PF0-OSC_IN; no longer U$4.PF0-OSC_IN
- net MCO_2: now also IC7.PA8; no longer U$5.PA8
- net N$1: now also IC5.R_S, R11.2; no longer IC7.R_S, R31.2
- net N$10: now also C12.1, IC1.PF1-OSC_OUT, Q1.2; no longer C31.1, Q2.2, U$2.PF1-OSC_OUT
- net N$11: now also C11.1, IC1.PF0-OSC_IN, Q1.1; no longer C30.1, Q2.1, U$2.PF0-OSC_IN
- net N$12: now also IC6.R_S, R12.2; no longer IC1.R_S, R32.2
- net N$13: now also C26.1, C29.1, C32.1, C34.1, IC6.V_ISOIN, IC6.V_ISOOUT; no longer C39.1, C42.1, C43.1, C44.1, IC1.V_ISOIN, IC1.V_ISOOUT
- net N$14: now also R7.1; no longer R33.1
- net N$15: now also LED7.A; no longer LED4.A
- net N$17: now also LED7.C, R21.2; no longer LED4.C, R14.2
- net N$18: now also R22.2; no longer R15.2
- net N$19: now also R8.1; no longer R34.1
- net N$2: now also C51.1, Q2.2, U$5.X2; no longer C1.1, Q1.2, U$3.X2
- net N$20: now also C47.1; no longer C46.1
- net N$22: now also IC1.PB1; no longer U$2.PB1
- net N$23: now also IC1.PB0, LED2.A; no longer LED5.A, U$2.PB0
- net N$24: now also R3.2; no longer R5.2
- net N$25: now also LED2.C, R4.2; no longer LED5.C, R6.2
- net N$26: now also IC4G$1.CANH, R10.1; no longer R36.1, U$1G$1.CANH
- net N$27: now also IC4G$1.CANL, R9.1; no longer R35.1, U$1G$1.CANL
- net N$28: now also JP4.1, R15.1; no longer JP3.1, R9.1
- net N$29: now also IC2.PB1, LED3.A; no longer LED2.A, U$4.PB1
- net N$3: now also C49.1, Q2.1, U$5.X1; no longer C2.1, Q1.1, U$3.X1
- net N$30: now also IC2.PB0, LED4.A; no longer LED6.A, U$4.PB0
- net N$31: now also LED3.C, R5.2; no longer LED2.C, R7.2
- net N$32: now also LED4.C, R6.2; no longer LED6.C, R8.2
- net N$33: now also C57.1, C58.+, R33.2, R34.2, U$5.DVDD, U$5.V33; no longer C6.1, C9.+, R1.2, R2.2, U$3.DVDD, U$3.V33
- net N$34: now also R33.1, U$5.PGANG; no longer R2.1, U$3.PGANG
- net N$35: now also R34.1, U$5.PSELF; no longer R1.1, U$3.PSELF
- net N$36: now also C55.1, R31.2, R32.2, U$5.RESET#; no longer C33.1, R16.2, R17.2, U$3.RESET#
- net N$37: now also U$5.DP0; no longer U$3.DP0
- net N$38: now also U$5.DM0; no longer U$3.DM0
- net N$39: now also C52.1, C53.1, C54.1, U$5.AVDD, U$5.AVDD2, U$5.AVDD3; no longer C3.1, C4.1, C5.1, U$3.AVDD, U$3.AVDD2, U$3.AVDD3
- net N$4: now also IC7.PB1, LED5.A; no longer LED3.A, U$5.PB1
- net N$40: now also R27.2, U$5.RREF; no longer R18.2, U$3.RREF
- net N$44: now also R36.2; no longer R19.2
- net N$48: now also JP3.1, R13.1; no longer JP6.1, R22.1
- net N$49: now also C30.1, R15.2, R16.2; no longer C37.1, R20.2, R9.2
- net N$5: now also IC11.WP, R28.2; no longer IC6.WP, R30.2
- net N$53: now also C28.1, R13.2, R14.2; no longer C41.1, R21.2, R22.2
- net N$56: now also IC7.PB8; no longer U$5.PB8
- net N$57: now also IC7.PB9; no longer U$5.PB9
- net N$59: now also R25.1; no longer R26.1
- net N$6: now also R23.1; no longer R24.1
- net N$63: now also C48.1; no longer C51.1
- net N$65: now also C25.1, C27.1, C31.1, C33.1, IC5.V_ISOIN, IC5.V_ISOOUT; no longer C59.1, C60.1, C61.1, C62.1, IC7.V_ISOIN, IC7.V_ISOOUT
- net N$7: now also IC7.PB0, LED6.A; no longer LED7.A, U$5.PB0
- net N$8: now also LED5.C, R19.2; no longer LED3.C, R12.2
- net N$9: now also LED6.C, R20.2; no longer LED7.C, R13.2
- net NRST: now also IC1.NRST, IC2.NRST, IC7.NRST, U$1.5; no longer U$2.NRST, U$4.NRST, U$5.NRST, U$8.5
- net SCL: now also IC12.SCL; no longer IC5.SCL
- net SDA: now also IC12.SDA; no longer IC5.SDA
- net SWCLK: now also IC1.PA14, IC2.PA14, IC7.PA14, U$1.2; no longer U$2.PA14, U$4.PA14, U$5.PA14, U$8.2
- net SWDIO: now also IC1.PA13, IC2.PA13, IC7.PA13, U$1.4; no longer U$2.PA13, U$4.PA13, U$5.PA13, U$8.4
- net USB0_DM: now also IC1.PA11, U$5.DM1; no longer U$2.PA11, U$3.DM1
- net USB0_DP: now also IC1.PA12, U$5.DP1; no longer U$2.PA12, U$3.DP1
- net USB1_DM: now also IC2.PA11, U$5.DM2; no longer U$3.DM2, U$4.PA11
- net USB1_DP: now also IC2.PA12, U$5.DP2; no longer U$3.DP2, U$4.PA12
- net USB2_DM: now also IC7.PA11, U$5.DM3; no longer U$3.DM3, U$5.PA11
- net USB2_DP: now also IC7.PA12, U$5.DP3; no longer U$3.DP3, U$5.PA12
- net USB3_DM: now also U$5.DM4; no longer U$3.DM4
- net USB3_DP: now also U$5.DP4; no longer U$3.DP4
- net VBAT: now also IC12.VBAT; no longer IC5.VBAT
