File: interface/Designs/OOBDpiCAN/pcb/sch/OOBDpiCAN.sch (EAGLE design)
At the start: 148 parts, among them IC1 STM32F042CT, IC10 MCP2551SO8, IC11 EEPROM24, IC12 DS3231, IC2 STM32F042CT, IC3 MCP2551SO8, IC4 MCP2551SO8, IC5 ADM3053M, IC6 ADM3053M, IC7 STM32F042CT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

Commit message: modification on component placing for OOBDpiCAN
Parts:
- removed C10, C43, C44, C9: 100nF, resistor:C-EUC0603
Connections:
- removed net SWCLK1: IC8.PA14
- removed net SWDIO1: IC8.PA13
- net +3V3: no longer C10.1, C43.1, C44.1, C9.1
- net GND: no longer C10.2, C43.2, C44.2, C9.2
- net SWCLK: now also IC8.PA14
- net SWDIO: now also IC8.PA13
Changed lines of the file:
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@@
 <part name="R17" library="resistor" deviceset="R-EU_" device="R0603" value="510R"/>
 <part name="+3V2" library="supply1" deviceset="+3V3" device=""/>
-<part name="C43" library="resistor" deviceset="C-EU" device="C0603" value="100nF"/>
 <part name="C41" library="resistor" deviceset="C-EU" device="C0603" value="100nF"/>
 <part name="C39" library="resistor" deviceset="C-EU" device="C0603" value="100nF"/>
@@
 <part name="R18" library="resistor" deviceset="R-EU_" device="R0603" value="510R"/>
 <part name="+3V4" library="supply1" deviceset="+3V3" device=""/>
-<part name="C44" library="resistor" deviceset="C-EU" device="C0603" value="100nF"/>
 <part name="C42" library="resistor" deviceset="C-EU" device="C0603" value="100nF"/>
 <part name="C40" library="resistor" deviceset="C-EU" device="C0603" value="100nF"/>
@@
 <part name="R1" library="resistor" deviceset="R-EU_" device="R0603" value="510R"/>
 <part name="+3V7" library="supply1" deviceset="+3V3" device=""/>
-<part name="C9" library="resistor" deviceset="C-EU" device="C0603" value="100nF"/>
 <part name="C7" library="resistor" deviceset="C-EU" device="C0603" value="100nF"/>
 <part name="C5" library="resistor" deviceset="C-EU" device="C0603" value="100nF"/>
@@
 <part name="R2" library="resistor" deviceset="R-EU_" device="R0603" value="510R"/>
 <part name="+3V9" library="supply1" deviceset="+3V3" device=""/>
-<part name="C10" library="resistor" deviceset="C-EU" device="C0603" value="100nF"/>
 <part name="C8" library="resistor" deviceset="C-EU" device="C0603" value="100nF"/>
 <part name="C6" library="resistor" deviceset="C-EU" device="C0603" value="100nF"/>
@@
 <instance part="R1" gate="G$1" x="83.82" y="177.8" rot="R90"/>
 <instance part="+3V7" gate="G$1" x="55.88" y="203.2"/>
-<instance part="C9" gate="G$1" x="78.74" y="223.52"/>
 <instance part="C7" gate="G$1" x="73.66" y="223.52"/>
 <instance part="C5" gate="G$1" x="68.58" y="223.52"/>
@@
 <instance part="R2" gate="G$1" x="83.82" y="48.26" rot="R90"/>
 <instance part="+3V9" gate="G$1" x="55.88" y="73.66"/>
-<instance part="C10" gate="G$1" x="78.74" y="93.98"/>
 <instance part="C8" gate="G$1" x="73.66" y="93.98"/>
 <instance part="C6" gate="G$1" x="68.58" y="93.98"/>
@@
 <wire x1="68.58" y1="215.9" x2="68.58" y2="213.36" width="0.1524" layer="91"/>
 <wire x1="68.58" y1="215.9" x2="73.66" y2="215.9" width="0.1524" layer="91"/>
-<pinref part="C9" gate="G$1" pin="2"/>
-<wire x1="73.66" y1="215.9" x2="78.74" y2="215.9" width="0.1524" layer="91"/>
-<wire x1="78.74" y1="215.9" x2="78.74" y2="218.44" width="0.1524" layer="91"/>
 <pinref part="C7" gate="G$1" pin="2"/>
 <wire x1="73.66" y1="218.44" x2="73.66" y2="215.9" width="0.1524" layer="91"/>
@@
 <junction x="63.5" y="215.9"/>
 <junction x="68.58" y="215.9"/>
-<junction x="73.66" y="215.9"/>
 </segment>
 <segment>
@@
 <wire x1="68.58" y1="86.36" x2="68.58" y2="83.82" width="0.1524" layer="91"/>
 <wire x1="68.58" y1="86.36" x2="73.66" y2="86.36" width="0.1524" layer="91"/>
-<pinref part="C10" gate="G$1" pin="2"/>
-<wire x1="73.66" y1="86.36" x2="78.74" y2="86.36" width="0.1524" layer="91"/>
-<wire x1="78.74" y1="86.36" x2="78.74" y2="88.9" width="0.1524" layer="91"/>
 <pinref part="C8" gate="G$1" pin="2"/>
 <wire x1="73.66" y1="88.9" x2="73.66" y2="86.36" width="0.1524" layer="91"/>
@@
 <junction x="63.5" y="86.36"/>
 <junction x="68.58" y="86.36"/>
-<junction x="73.66" y="86.36"/>
 </segment>
 <segment>
@@
 <pinref part="C7" gate="G$1" pin="1"/>
 <wire x1="73.66" y1="228.6" x2="73.66" y2="226.06" width="0.1524" layer="91"/>
-<pinref part="C9" gate="G$1" pin="1"/>
-<wire x1="78.74" y1="228.6" x2="78.74" y2="226.06" width="0.1524" layer="91"/>
 <junction x="63.5" y="228.6"/>
 <junction x="68.58" y="228.6"/>
 <junction x="73.66" y="228.6"/>
-<junction x="78.74" y="228.6"/>
 </segment>
 <segment>
@@
 <pinref part="C8" gate="G$1" pin="1"/>
 <wire x1="73.66" y1="99.06" x2="73.66" y2="96.52" width="0.1524" layer="91"/>
-<pinref part="C10" gate="G$1" pin="1"/>
-<wire x1="78.74" y1="99.06" x2="78.74" y2="96.52" width="0.1524" layer="91"/>
 <junction x="63.5" y="99.06"/>
 <junction x="68.58" y="99.06"/>
 <junction x="73.66" y="99.06"/>
-<junction x="78.74" y="99.06"/>
 </segment>
 <segment>
@@
 <instance part="R17" gate="G$1" x="83.82" y="177.8" rot="R90"/>
 <instance part="+3V2" gate="G$1" x="55.88" y="203.2"/>
-<instance part="C43" gate="G$1" x="78.74" y="223.52"/>
 <instance part="C41" gate="G$1" x="73.66" y="223.52"/>
 <instance part="C39" gate="G$1" x="68.58" y="223.52"/>
@@
 <instance part="R18" gate="G$1" x="83.82" y="48.26" rot="R90"/>
 <instance part="+3V4" gate="G$1" x="55.88" y="73.66"/>
-<instance part="C44" gate="G$1" x="78.74" y="93.98"/>
 <instance part="C42" gate="G$1" x="73.66" y="93.98"/>
 <instance part="C40" gate="G$1" x="68.58" y="93.98"/>
@@
 <wire x1="68.58" y1="215.9" x2="68.58" y2="213.36" width="0.1524" layer="91"/>
 <wire x1="68.58" y1="215.9" x2="73.66" y2="215.9" width="0.1524" layer="91"/>
-<pinref part="C43" gate="G$1" pin="2"/>
-<wire x1="73.66" y1="215.9" x2="78.74" y2="215.9" width="0.1524" layer="91"/>
-<wire x1="78.74" y1="215.9" x2="78.74" y2="218.44" width="0.1524" layer="91"/>
 <pinref part="C41" gate="G$1" pin="2"/>
 <wire x1="73.66" y1="218.44" x2="73.66" y2="215.9" width="0.1524" layer="91"/>
@@
 <junction x="63.5" y="215.9"/>
 <junction x="68.58" y="215.9"/>
-<junction x="73.66" y="215.9"/>
 </segment>
 <segment>
@@
 <wire x1="68.58" y1="86.36" x2="68.58" y2="83.82" width="0.1524" layer="91"/>
 <wire x1="68.58" y1="86.36" x2="73.66" y2="86.36" width="0.1524" layer="91"/>
-<pinref part="C44" gate="G$1" pin="2"/>
-<wire x1="73.66" y1="86.36" x2="78.74" y2="86.36" width="0.1524" layer="91"/>
-<wire x1="78.74" y1="86.36" x2="78.74" y2="88.9" width="0.1524" layer="91"/>
 <pinref part="C42" gate="G$1" pin="2"/>
 <wire x1="73.66" y1="88.9" x2="73.66" y2="86.36" width="0.1524" layer="91"/>
@@
 <junction x="63.5" y="86.36"/>
 <junction x="68.58" y="86.36"/>
-<junction x="73.66" y="86.36"/>
 </segment>
 <segment>
@@
 <pinref part="C41" gate="G$1" pin="1"/>
 <wire x1="73.66" y1="228.6" x2="73.66" y2="226.06" width="0.1524" layer="91"/>
-<pinref part="C43" gate="G$1" pin="1"/>
-<wire x1="78.74" y1="228.6" x2="78.74" y2="226.06" width="0.1524" layer="91"/>
 <junction x="63.5" y="228.6"/>
 <junction x="68.58" y="228.6"/>
 <junction x="73.66" y="228.6"/>
-<junction x="78.74" y="228.6"/>
 </segment>
 <segment>
@@
 <pinref part="C42" gate="G$1" pin="1"/>
 <wire x1="73.66" y1="99.06" x2="73.66" y2="96.52" width="0.1524" layer="91"/>
-<pinref part="C44" gate="G$1" pin="1"/>
-<wire x1="78.74" y1="99.06" x2="78.74" y2="96.52" width="0.1524" layer="91"/>
 <junction x="63.5" y="99.06"/>
 <junction x="68.58" y="99.06"/>
 <junction x="73.66" y="99.06"/>
-<junction x="78.74" y="99.06"/>
 </segment>
 <segment>
@@
 <label x="200.66" y="195.58" size="1.27" layer="95" xref="yes"/>
 </segment>
+<segment>
+<pinref part="IC8" gate="G$1" pin="PA13"/>
+<wire x1="180.34" y1="66.04" x2="200.66" y2="66.04" width="0.1524" layer="91"/>
+<label x="200.66" y="66.04" size="1.27" layer="95" xref="yes"/>
+</segment>
 </net>
 <net name="SWCLK" class="0">
@@
 <label x="200.66" y="193.04" size="1.27" layer="95" xref="yes"/>
 </segment>
+<segment>
+<pinref part="IC8" gate="G$1" pin="PA14"/>
+<wire x1="200.66" y1="63.5" x2="180.34" y2="63.5" width="0.1524" layer="91"/>
+<label x="200.66" y="63.5" size="1.27" layer="95" xref="yes"/>
+</segment>
 </net>
 <net name="N$4" class="0">
@@
 </segment>
 </net>
-<net name="SWDIO1" class="0">
-<segment>
-<pinref part="IC8" gate="G$1" pin="PA13"/>
-<wire x1="180.34" y1="66.04" x2="200.66" y2="66.04" width="0.1524" layer="91"/>
-<label x="200.66" y="66.04" size="1.27" layer="95" xref="yes"/>
-</segment>
-</net>
-<net name="SWCLK1" class="0">
-<segment>
-<pinref part="IC8" gate="G$1" pin="PA14"/>
-<wire x1="200.66" y1="63.5" x2="180.34" y2="63.5" width="0.1524" layer="91"/>
-<label x="200.66" y="63.5" size="1.27" layer="95" xref="yes"/>
-</segment>
-</net>
 <net name="N$15" class="0">
 <segment>
@@
 <wire x1="109.22" y1="137.16" x2="109.22" y2="139.7" width="0.1524" layer="91"/>
 <pinref part="R29" gate="G$1" pin="2"/>
-<label x="109.22" y="137.16" size="1.778" layer="95"/>
+<label x="127" y="137.16" size="1.27" layer="95" xref="yes"/>
+<wire x1="109.22" y1="137.16" x2="127" y2="137.16" width="0.1524" layer="91"/>
+<junction x="109.22" y="137.16"/>
 </segment>
 </net>
@@
 <wire x1="101.6" y1="134.62" x2="119.38" y2="134.62" width="0.1524" layer="91"/>
 <pinref part="R30" gate="G$1" pin="2"/>
-<label x="109.22" y="134.62" size="1.778" layer="95"/>
+<label x="127" y="134.62" size="1.27" layer="95" xref="yes"/>
+<wire x1="119.38" y1="134.62" x2="127" y2="134.62" width="0.1524" layer="91"/>
+<junction x="119.38" y="134.62"/>
 </segment>
 </net>
@@
 </sheet>
 </sheets>
+<errors>
+</errors>
 </schematic>
 </drawing>

Commit message: add initial version of OOBDpiZero rearrange Eagle library files
Parts:
- removed C11, C12: 18pF, resistor:C-EUC0603
- removed C17, C18: 10u, rcl:C-EUC0805K
- removed Q1: 16MHz, crystal:CRYSTALSM49
- removed R38: 0R, rcl:R-EU_R0603
- removed R39: 0R, resistor:R-EU_R0603
- added C10, C9: 10n, rcl:C-EUC0603K
- R37: device rcl:R-EU_R0603 -> rcl:R-EU_0207/10
Connections:
- removed net MC0_1: IC7.PF0-OSC_IN, R38.1
- removed net MCO_0: R37.1
- removed net MCO_1: IC2.PF0-OSC_IN
- removed net MCO_2: IC8.PF0-OSC_IN, R39.2
- removed net N$10: C12.1, IC1.PF1-OSC_OUT, Q1.2
- removed net N$11: C11.1, IC1.PF0-OSC_IN, Q1.1
- removed net N$43: IC1.PA8, R37.2
- removed net N$45: IC2.PA8, R38.2
- removed net N$46: IC7.PA8, R39.1
- net +3V3: now also C10.1, C9.1; no longer C17.1, C18.1
- net GND: now also C10.2, C9.2, R37.2; no longer C11.2, C12.2, C17.2, C18.2
- net GNDA: now also R37.1
Other:
- note removed: "optional"
- moved on the sheet: R37
