File: interface/Designs/OOBDpiZero/pcb/OOBDpiZero.sch (EAGLE design)
At the start: 132 parts, among them IC1 EEPROM24, IC100 LM1117MPX-3.3, IC2 DS3231, Q1 12MHz, U1 MAX98357, U100 SY6280, U101 SN65HVD230(SO8), U102 SN65HVD230(SO8), U2 MP1482

Commit message: - DRC with "PCB-POOL HighSpec.dru" without errors - One signal "SDIO" not routed completely
Parts:
- GPIO: value PIZERO_THROUGH_HOLE -> OOBDpiZero
Connections:
- removed net HS-CAN_RS: GPIO.35
- removed net MS-CAN_RS: GPIO.36
Changed lines of the file:
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@@
 <part name="GND38" library="supply1" deviceset="GND" device="" value="GND"/>
 <part name="+3V10" library="supply1" deviceset="+3V3" device=""/>
-<part name="GPIO" library="pizero" deviceset="PIZERO_THROUGH_HOLE" device=""/>
+<part name="GPIO" library="pizero" deviceset="PIZERO_THROUGH_HOLE" device="" value="OOBDpiZero"/>
 <part name="U1" library="microbuilder" deviceset="AUDIOAMP_MAX98357" device="" value="MAX98357"/>
 <part name="U$100" library="micro-stm_v3" deviceset="STM32F042C*T" device=""/>
@@
 </segment>
 </net>
-<net name="HS-CAN_RS" class="0">
-<segment>
-<pinref part="GPIO" gate="1" pin="35"/>
-<wire x1="233.68" y1="104.14" x2="215.9" y2="104.14" width="0.1524" layer="91"/>
-<label x="215.9" y="104.14" size="1.27" layer="95" rot="R180" xref="yes"/>
-</segment>
-</net>
-<net name="MS-CAN_RS" class="0">
-<segment>
-<pinref part="GPIO" gate="1" pin="36"/>
-<wire x1="248.92" y1="104.14" x2="266.7" y2="104.14" width="0.1524" layer="91"/>
-<label x="266.7" y="104.14" size="1.27" layer="95" xref="yes"/>
-</segment>
-</net>
